File: AK4493-v1.64_25.sch (EAGLE design)
At the start: 138 parts, among them IC1 LT3042, IC2 AK4493, IC3 AK4493, IC4 LT3042, IC4A SN74ABT273DBR, IC5 LT3042, IC6 LT3042, IC7 LT3042, IC8 LT3042, J15 XR2A-0811-N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

Commit message: Updating board for breakout boards
Parts:
- added J21, J22: (no value), SparkFun-Connectors:CONN_10"
Connections:
- new net N$3: IC4A.GND, J21.1
- new net N$4: IC4A.3Q, J21.5
- new net N$5: IC4A.7Q, J22.5
- net +3V3: now also J22.1
- net BCLK: now also J21.3, J22.3
- net DATA: now also J21.7, J22.7
- net DGND: now also J21.4, J22.4; no longer IC4A.GND
- net LRCK: now also J21.8, J22.8
- net MCLK: now also J22.10
- net N$1: now also J21.10
- net N$23: now also J22.2
- net N$24: now also J22.6
- net N$25: now also J22.9
- net N$30: now also J21.2
- net N$31: now also J21.6
- net N$32: now also J21.9
Other:
- moved on the sheet: C10A2, C11B, C12A2, C13B, C14A2, C15B, C16A2, C17B, C18B, C18D, C18E, C18F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
