File: AK4493-v1.64_26.brd (EAGLE design)
At the start: 89.9 x 99.5 mm, 140 parts, among them IC1 LT3042, IC2 AK4493, IC3 AK4493, IC4 LT3042, IC4A SN74ABT273DBR, IC5 LT3042, IC6 LT3042, IC7 LT3042, IC8 LT3042, J15 XR2A-0811-N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

Commit message: Progress
Parts:
- moved R4A 0.07 mm to (57.6, 12.0)
- moved R4B 0.07 mm to (15.2, 29.1)
Routing:
- net MCLK: track 154.6 -> 220.4 mm
- net N$23: track 58.5 -> 82.3 mm
- net N$31: track 62.0 -> 78.1 mm
- net N$24: track 63.3 -> 78.0 mm
- net N$32: track 60.0 -> 72.2 mm
- net N$25: track 74.0 -> 82.8 mm
- net N$30: track 75.3 -> 83.2 mm
- net SDA0: track 184.2 -> 179.6 mm
- net DIF0: track 124.5 -> 120.0 mm
- net DIF1: track 122.0 -> 117.4 mm
- net SCL0: track 183.2 -> 178.7 mm
- net PDN: track 225.7 -> 221.5 mm

Commit message: Getting closer
Parts:
- moved J3 86.9 mm to (44.9, 18.4), turned to 270 degrees
- moved R20 83.9 mm to (40.7, 13.3), turned to 180 degrees
- moved C1A 83.5 mm to (40.7, 21.0), turned to 0 degrees
- moved R10 82.5 mm to (40.7, 15.9), turned to 180 degrees
- moved R5A 81.2 mm to (40.7, 18.4), turned to 0 degrees
- moved C18E 4.47 mm to (13.6, 81.9)
- moved C19E 4.47 mm to (25.7, 77.1)
- moved C20E 4.47 mm to (17.3, 90.7)
- moved C21E 4.47 mm to (13.6, 87.1)
- moved IC8 4.47 mm to (20.3, 84.0)
- moved J20 4.47 mm to (24.1, 87.8)
- moved R6E 4.47 mm to (27.0, 86.3)
- moved R7E 4.47 mm to (27.1, 81.2)
- moved R8E 4.47 mm to (23.2, 90.8)
- moved C3A 2.17 mm to (51.2, 24.6), turned to 225 degrees
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Routing:
- net PDN: track 221.5 -> 56.6 mm, vias 2 -> 1
- net SCL0: track 178.7 -> 60.7 mm, vias 2 -> 1
- net SDA0: track 179.6 -> 67.5 mm, vias 2 -> 0
- net DIF0: track 120.0 -> 54.6 mm, vias 0 -> 1
- net DIF1: track 117.4 -> 61.8 mm, vias 0 -> 1
- net +3V3: track 252.5 -> 215.0 mm
- net +5V/3: track 53.9 -> 58.8 mm, vias 0 -> 3
- net +5V/1: track 102.1 -> 105.0 mm
- net +5V/5: track 89.0 -> 87.8 mm
- net VCC/2: track 85.6 -> 86.8 mm

Commit message: Finished design and generated gerbers
Routing:
- net +5V/3: track 58.8 -> 60.8 mm
- net VCC/3: track 82.4 -> 81.2 mm
