File: AK4493-Combi.brd (EAGLE design)
At the start: 178 x 151.3 mm, 220 parts, among them IC1 LT3042, IC2 AK4493, IC3 AK4493, IC4 LT3042, IC4A SN74ABT273DBR, IC5 LT3042, IC6 LT3042, IC7 LT3042, IC8 LT3042, J15 XR2A-0811-N, J16 XR2A-0811-N, J17 XR2A-0811-N, J18 XR2A-0811-N, J19 XR2A-0811-N, J20 XR2A-0811-N, J26 SJ-63033A, J27 1935161

Commit message: Progress
Parts:
- moved C18C 110.2 mm to (170.2, 126.9)
- moved C20C 110.2 mm to (165.1, 126.9)
- moved R7C 110.2 mm to (171.0, 140.3)
- moved R8C 110.2 mm to (161.4, 136.4)
- moved C19C 110.2 mm to (175.0, 138.9)
- moved C21C 110.2 mm to (161.4, 130.5)
- moved IC4 110.2 mm to (168.1, 133.5)
- moved J16 110.2 mm to (164.3, 137.4)
- moved R6C 110.2 mm to (165.9, 140.2)
- moved U$1 99.8 mm to (59.2, 130.8), turned to 270 degrees
- moved R8A 79.0 mm to (152.2, 130.6), turned to 270 degrees
- moved C20A 78.0 mm to (152.1, 136.5), turned to 270 degrees
- moved J15 73.6 mm to (149.2, 129.6), turned to 90 degrees
- moved R6A 71.8 mm to (147.6, 126.8), turned to 180 degrees
- moved C21A 71.0 mm to (148.4, 140.1), turned to 0 degrees
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Connections:
- net N$79: now also C11O.1; no longer C12O.1
- net N$80: now also C12O.1; no longer C11O.1
- net N$87: now also C13O.1; no longer C14O.1
- net N$88: now also C14O.1; no longer C13O.1
Routing:
- net +240VDC: track 135.2 -> 326.7 mm
- net +3V3: track 118.0 -> 28.9 mm, vias 3 -> 0
- net +5V/3: track 2.88 -> 61.3 mm
- net DIF1: track 54.6 -> 7.67 mm, vias 1 -> 0
- net 66.3VAC/2: track 109.2 -> 152.6 mm
- net DIF0: track 48.7 -> 8.38 mm, vias 1 -> 0
- net N$65: track 0.00 -> 40.3 mm
- net SDA0: track 61.9 -> 23.7 mm
- net SCL0: track 54.3 -> 20.2 mm
- net MCLK: track 80.7 -> 113.6 mm
- net PDN: track 50.8 -> 20.4 mm
- net N$64: track 6.00 -> 35.6 mm
- net 6.3_VAC_ORG: track 84.3 -> 107.4 mm
- net N$90: track 17.5 -> 36.3 mm
- net N$79: track 17.5 -> 36.3 mm
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- added copper zone on layer 1, net AGND

Commit message: Progress
Parts:
- removed J3: (no value), Dual Mono Amp Library:1X07
- added C6, C7: 0.1 uF, Hifi Nutube DAC 44:C0603
- added D9: 1A/40V/500mV, SparkFun-DiscreteSemi:SMA-DIODE
- added R1: 5k, Hifi Nutube DAC 44:R0603
- added X2: JST-XH-07-PIN-LONG-PAD, Rembrandt Electronics - JST XH Connectors v1-0:JST-XH-07-PACKAGE-LONG-PAD
- moved R20 82.7 mm to (70.8, 124.2), turned to 0 degrees
- moved R10 81.4 mm to (70.8, 121.7), turned to 0 degrees
- moved R5A 80.2 mm to (70.8, 119.2), turned to 180 degrees
- moved C1A 79.1 mm to (70.8, 116.6), turned to 180 degrees
- moved C26B 1.41 mm to (105.7, 124.6)
- moved C3B 1.41 mm to (96.3, 123.7)
- moved C5B 1.41 mm to (92.6, 119.1)
- moved LDO8 1.41 mm to (103.4, 122.2)
- moved R4B 1.41 mm to (92.2, 115.9)
- moved U$1 0.20 mm to (59.2, 130.6)
Connections:
- new net N$15: D9.A, U$1.VUSB
- new net N$39: D9.C, U$1.VIN
- new net ROT_A: C6.1, U$1.3-LRCLK2, X2.1
- new net ROT_B: C7.2, U$1.5-IN2, X2.3
- new net ROT_LEDB: U$1.23-A9/CRX1/CCLK1, X2.4
- new net ROT_LEDG: U$1.22-A8/CTX1, X2.5
- new net ROT_LEDR: U$1.19-A5/SCL0, X2.6
- new net ROT_SW: R1.2, U$1.4-BCLK2, X2.2
- net +3V3: no longer J3.4
- net AGND: now also IC2.P$1, IC2.P$10, IC2.P$11, IC2.P$12, IC2.P$13, IC2.P$14, IC2.P$15, IC2.P$16, IC2.P$17, IC2.P$18, IC2.P$19, IC2.P$2, IC2.P$20, IC2.P$21, IC2.P$22, IC2.P$23, IC2.P$24, IC2.P$25, IC2.P$3, IC2.P$4, IC2.P$5, IC2.P$6, IC2.P$7, IC2.P$8, IC2.P$9, IC3.P$1, IC3.P$10, IC3.P$11, IC3.P$12, IC3.P$13, IC3.P$14, IC3.P$15, IC3.P$16, IC3.P$17, IC3.P$18, IC3.P$19, IC3.P$2, IC3.P$20, IC3.P$21, IC3.P$22, IC3.P$23, IC3.P$24, IC3.P$25, IC3.P$3, IC3.P$4, IC3.P$5, IC3.P$6, IC3.P$7, IC3.P$8, IC3.P$9
- net DGND: now also C6.2, C7.1, R1.1, U$1.GND1, U$1.GND2, U$1.GND3, X2.7; no longer IC2.P$1, IC2.P$10, IC2.P$11, IC2.P$12, IC2.P$13, IC2.P$14, IC2.P$15, IC2.P$16, IC2.P$17, IC2.P$18, IC2.P$19, IC2.P$2, IC2.P$20, IC2.P$21, IC2.P$22, IC2.P$23, IC2.P$24, IC2.P$25, IC2.P$3, IC2.P$4, IC2.P$5, IC2.P$6, IC2.P$7, IC2.P$8, IC2.P$9, IC3.P$1, IC3.P$10, IC3.P$11, IC3.P$12, IC3.P$13, IC3.P$14, IC3.P$15, IC3.P$16, IC3.P$17, IC3.P$18, IC3.P$19, IC3.P$2, IC3.P$20, IC3.P$21, IC3.P$22, IC3.P$23, IC3.P$24, IC3.P$25, IC3.P$3, IC3.P$4, IC3.P$5, IC3.P$6, IC3.P$7, IC3.P$8, IC3.P$9, J3.5
- net DIF0: now also U$1.1-TX1; no longer J3.6
- net DIF1: now also U$1.2-OUT2; no longer J3.7
- net PDN: now also U$1.0-RX1; no longer J3.1
- net SCL0: now also U$1.16-A2/RX4/SCL1; no longer J3.2
- net SDA0: now also U$1.17-A3/TX4/SDA1; no longer J3.3
Routing:
- net PDN: track 20.4 -> 195.2 mm, vias 1 -> 2
- net +3V3: track 28.9 -> 180.4 mm, vias 0 -> 6
- net SDA0: track 23.7 -> 136.2 mm
- net SCL0: track 20.2 -> 127.5 mm
- net VCC/1: track 341.4 -> 435.5 mm
- net +5V/4: track 2.88 -> 65.5 mm
- net +5V/2: track 72.6 -> 116.9 mm
- net +5V/1: track 61.0 -> 104.6 mm
- net N$39: track 0.00 -> 6.52 mm
- net N$15: track 0.00 -> 4.71 mm
- net MCLK: track 113.6 -> 118.2 mm
- net ROT_SW: track 0.00 -> 2.97 mm
- net ROT_B: track 0.00 -> 2.97 mm
- net ROT_A: track 0.00 -> 2.97 mm
- net 66.3VAC/1: track 134.6 -> 132.4 mm
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
Commit message: Progress
Parts:
- removed C8P, C9P: UCY2E220MPD1TD, UCY2E220MPD1TD:CAPPRD500W60D1025H1750
- removed X2: JST-XH-07-PIN-LONG-PAD, Rembrandt Electronics - JST XH Connectors v1-0:JST-XH-07-PACKAGE-LONG-PAD
- added U1: AZ1117H-5.0TRE1, AZ1117H-5.0TRE1:SOT230P700X180-4N
- added X1: JST-XH-07-PIN-ROUND-PAD, Rembrandt Electronics - JST XH Connectors v1-0:JST-XH-07-PACKAGE-ROUND-PAD
- added X4: JST-XH-04-PIN-ROUND-PAD, Rembrandt Electronics - JST XH Connectors v1-0:JST-XH-04-PACKAGE-ROUND-PAD
- moved C19E 68.7 mm to (130.4, 91.2)
- moved R7E 68.7 mm to (126.3, 92.6)
- moved R8E 68.7 mm to (116.7, 88.7)
- moved C18E 68.7 mm to (125.6, 79.2)
- moved C20E 68.7 mm to (116.8, 82.8)
- moved C21E 68.7 mm to (120.4, 79.2)
- moved IC8 68.7 mm to (123.5, 85.8)
- moved J20 68.7 mm to (119.7, 89.7)
- moved R6E 68.7 mm to (121.2, 92.5)
- moved R6B 19.1 mm to (49.4, 66.0), turned to 270 degrees
- moved R8B 18.7 mm to (53.2, 61.5), turned to 0 degrees
- moved R7B 17.4 mm to (49.3, 71.1), turned to 270 degrees
- moved J17 16.8 mm to (52.2, 64.4), turned to 180 degrees
- moved C19B 16.1 mm to (50.7, 75.1), turned to 180 degrees
- moved C20B 14.8 mm to (59.1, 61.5), turned to 0 degrees
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Connections:
- removed net 6.3_VAC_BRN: C9P.1, IN.1
- removed net 6.3_VAC_ORG: C8P.1, IN.2
- net 66.3VAC/1: now also IN.1; no longer C9P.2
- net 66.3VAC/2: now also IN.2; no longer C8P.2
- net DGND: now also U1.1, X1.7, X4.4; no longer X2.7
- net N$39: now also U1.2, U1.4, X4.3
- net ROT_A: now also X1.1; no longer X2.1
- net ROT_B: now also X1.3; no longer X2.3
- net ROT_LEDB: now also X1.4; no longer X2.4
- net ROT_LEDG: now also X1.5; no longer X2.5
- net ROT_LEDR: now also X1.6; no longer X2.6
- net ROT_SW: now also X1.2; no longer X2.2
- net SCL0: now also X4.1
- net SDA0: now also X4.2
- net VCC/1: now also U1.3
Routing:
- net DIF0: track 8.38 -> 173.2 mm, vias 0 -> 2
- net 66.3VAC/1: track 132.4 -> 294.7 mm
- net DIF1: track 7.67 -> 168.6 mm, vias 0 -> 2
- net 66.3VAC/2: track 152.6 -> 313.0 mm
- net VCC/1: track 435.5 -> 563.3 mm
- net 6.3_VAC_ORG: track 107.4 -> 0.00 mm
- net 6.3_VAC_BRN: track 99.9 -> 0.00 mm, vias 3 -> 0
- net N$39: track 6.52 -> 83.5 mm
- net PDN: track 195.2 -> 152.9 mm, vias 2 -> 3
- net SDA0: track 136.2 -> 170.7 mm
- net ROT_B: track 2.97 -> 35.3 mm
- net SCL0: track 127.5 -> 157.0 mm, vias 1 -> 3
- net ROT_SW: track 2.97 -> 31.7 mm
- net ROT_LEDR: track 0.00 -> 26.9 mm
- net MCLK: track 118.2 -> 144.2 mm
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