File: AK4493-Combi.sch (EAGLE design)
At the start: 220 parts, among them IC1 LT3042, IC2 AK4493, IC3 AK4493, IC4 LT3042, IC4A SN74ABT273DBR, IC5 LT3042, IC6 LT3042, IC7 LT3042, IC8 LT3042, J15 XR2A-0811-N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

Commit message: Progress
Connections:
- net N$79: now also C11O.+; no longer C12O.+
- net N$80: now also C12O.+; no longer C11O.+
- net N$87: now also C13O.+; no longer C14O.+
- net N$88: now also C14O.+; no longer C13O.+
Other:
- moved on the sheet: C11O, C12O, C13O, C14O, R11O, R12O, R14O, R16O, R18O, R19O, R20O, R21O

Commit message: Progress
Parts:
- removed J3: (no value), Dual Mono Amp Library:CONN_07
- added C6, C7: 0.1 uF, Hifi Nutube DAC 44:C0603
- added D9: 1A/40V/500mV, SparkFun-DiscreteSemi:DIODE-SCHOTTKY-SS14
- added R1: 5k, Hifi Nutube DAC 44:R-US_R0603
- added X2: JST-XH-07-PIN-LONG-PAD, Rembrandt Electronics - JST XH Connectors v1-0:JST-XH-07-PIN-LONG-PAD
Connections:
- new net N$15: D9.A, U$1.VUSB
- new net N$39: D9.C, U$1.VIN
- new net ROT_A: C6.1, U$1.3-LRCLK2, X2-1.S
- new net ROT_B: C7.2, U$1.5-IN2, X2-3.S
- new net ROT_LEDB: U$1.23-A9/CRX1/MCLK1, X2-4.S
- new net ROT_LEDG: U$1.22-A8/CTX1, X2-5.S
- new net ROT_LEDR: U$1.19-A5/SCL0, X2-6.S
- new net ROT_SW: R1.2, U$1.4-BCLK1, X2-2.S
- net +3V3: no longer J3.4
- net DGND: now also C6.2, C7.1, R1.1, U$1.GND1, U$1.GND2, U$1.GND3, X2-7.S; no longer J3.5
- net DIF0: now also U$1.1-TX1/CTX2; no longer J3.6
- net DIF1: now also U$1.2-OUT2; no longer J3.7
- net PDN: now also U$1.0-RX1/CRX2; no longer J3.1
- net SCL0: now also U$1.16-A2/RX4/SCL1; no longer J3.2
- net SDA0: now also U$1.17-A3/TX4/SDA1; no longer J3.3

Commit message: Progress
Parts:
- removed C8P, C9P: UCY2E220MPD1TD, UCY2E220MPD1TD:UCY2E220MPD1TD
- removed X2: JST-XH-07-PIN-LONG-PAD, Rembrandt Electronics - JST XH Connectors v1-0:JST-XH-07-PIN-LONG-PAD
- added U1: AZ1117H-5.0TRE1, AZ1117H-5.0TRE1:AZ1117H-5.0TRE1
- added X1: JST-XH-07-PIN-ROUND-PAD, Rembrandt Electronics - JST XH Connectors v1-0:JST-XH-07-PIN-ROUND-PAD
- added X4: JST-XH-04-PIN-ROUND-PAD, Rembrandt Electronics - JST XH Connectors v1-0:JST-XH-04-PIN-ROUND-PAD
Connections:
- removed net 6.3_VAC_BRN: C9P.+, IN.1
- removed net 6.3_VAC_ORG: C8P.+, IN.2
- net 66.3VAC/1: now also IN.1; no longer C9P.-
- net 66.3VAC/2: now also IN.2; no longer C8P.-
- net DGND: now also U1.ADJ/GND, X1-7.S, X4-4.S; no longer X2-7.S
- net N$39: now also U1.OUTPUT, U1.VOUT, X4-3.S
- net ROT_A: now also X1-1.S; no longer X2-1.S
- net ROT_B: now also X1-3.S; no longer X2-3.S
- net ROT_LEDB: now also X1-4.S; no longer X2-4.S
- net ROT_LEDG: now also X1-5.S; no longer X2-5.S
- net ROT_LEDR: now also X1-6.S; no longer X2-6.S
- net ROT_SW: now also X1-2.S; no longer X2-2.S
- net SCL0: now also X4-1.S
- net SDA0: now also X4-2.S
- net VCC/1: now also U1.INPUT
Other:
- moved on the sheet: C1, C1P, C1P1, C2, C2P, C2P1, C3, C3P, C3P1, C4, C4P, C5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
