File: AK4493_Breakout_2.brd (EAGLE design)
At the start: 21.9 x 21.9 mm, 15 parts, among them IC2 AK4493

Commit message: Progress
Parts:
- moved IC2 0.72 mm to (10.4, 10.4)
- moved C14A1 0.72 mm to (16.9, 11.4)
- moved C16A1 0.72 mm to (16.8, 9.53)
- moved C10A1 0.72 mm to (11.8, 4.29)
- moved C12A1 0.72 mm to (14.7, 5.17)
- moved SMUTE1 0.72 mm to (5.19, 11.2)
- moved C6A1 0.72 mm to (11.9, 16.6)
- moved C8A1 0.72 mm to (14.7, 15.7)
- moved DIF1 0.72 mm to (6.49, 6.49)
- moved J8 0.72 mm to (1.56, 1.56)
- moved C2A1 0.72 mm to (6.20, 15.7)
- moved J5 0.72 mm to (19.3, 1.56)
- moved J7 0.72 mm to (1.56, 19.3)
- moved C4A1 0.72 mm to (8.97, 17.1)
- moved J6 0.72 mm to (19.3, 19.3)
Connections:
- new net AGND: C10A1.2, C10A1.3, C12A1.2, C12A1.3, C14A1.2, C14A1.3, C16A1.2, C16A1.3, C4A1.2, C4A1.3, C6A1.2, C6A1.3, C8A1.2, C8A1.3, IC2.21, IC2.22, IC2.29, IC2.30, IC2.31, IC2.32, IC2.39, IC2.40, IC2.45, IC2.P$1, IC2.P$10, IC2.P$17, IC2.P$18, IC2.P$2, IC2.P$25, IC2.P$4, IC2.P$6, IC2.P$8, J5.3, J6.2, J6.7
- net DGND: now also C2A1.3; no longer C10A1.2, C10A1.DGND, C12A1.2, C12A1.DGND, C14A1.2, C14A1.DGND, C16A1.2, C16A1.DGND, C2A1.DGND, C4A1.2, C4A1.DGND, C6A1.2, C6A1.DGND, C8A1.2, C8A1.DGND, IC2.21, IC2.22, IC2.24, IC2.29, IC2.30, IC2.31, IC2.32, IC2.39, IC2.40, IC2.45, IC2.P$1, IC2.P$10, IC2.P$11, IC2.P$12, IC2.P$13, IC2.P$14, IC2.P$15, IC2.P$16, IC2.P$17, IC2.P$18, IC2.P$19, IC2.P$2, IC2.P$20, IC2.P$21, IC2.P$22, IC2.P$23, IC2.P$24, IC2.P$25, IC2.P$3, IC2.P$4, IC2.P$5, IC2.P$6, IC2.P$7, IC2.P$8, IC2.P$9, J5.3, J6.2, J6.7
Routing:
- added copper zone on layer 1, net AGND
- added copper zone on layer 16, net AGND
Other:
- board size 21.9 x 21.9 mm -> 20.9 x 20.9 mm
- board text added: "AGND AORN VDDR VDDL AOLN AGND"
- board text added: "VCMR AGND VREFHR +3.3V DIF1 DIF0"
- board text removed: "DGND AORN VDDR VDDL AOLN DGND"
- board text removed: "VCMR DGND VREFHR +3.3V DIF1 DIF0"
