File: AK4493_Breakout_2.sch (EAGLE design)
At the start: 15 parts, among them IC2 AK4493

Commit message: Progress
Connections:
- new net AGND: C10A1.2, C12A1.2, C14A1.2, C16A1.2, C4A1.2, C6A1.2, C8A1.2, IC2.AVSS, IC2.VREFLL, IC2.VREFLL2, IC2.VREFLR, IC2.VREFLR2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
- net DGND: no longer C10A1.2, C12A1.2, C14A1.2, C16A1.2, C4A1.2, C6A1.2, C8A1.2, IC2.AVSS, IC2.NC, IC2.VREFLL, IC2.VREFLL2, IC2.VREFLR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
