File: AK4493-Combi2.brd (EAGLE design)
At the start: 178 x 151.3 mm, 224 parts, among them IC1 LT3042, IC3 AK4493, IC4 LT3042, IC4A SN74ABT273DBR, IC5 LT3042, IC6 LT3042, IC7 LT3042, IC8 LT3042, IC9 AK4493, J15 XR2A-0811-N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

Commit message: Progress
Routing:
- net N$32: track 22.6 -> 38.2 mm
- net N$23: track 26.7 -> 38.9 mm
- net N$31: track 25.8 -> 38.0 mm
- net SDA0: track 170.5 -> 159.5 mm
- net MCLK: track 141.7 -> 131.1 mm
- net N$91: track 23.0 -> 32.9 mm
- net N$116: track 23.1 -> 32.9 mm
- net N$24: track 28.7 -> 38.5 mm
- net SCL0: track 152.2 -> 145.1 mm
- net +3V3: track 162.1 -> 158.6 mm, vias 9 -> 8
- net VCC/1: track 542.1 -> 539.6 mm
- net PDN: track 152.3 -> 150.1 mm
- net DIF1: track 238.9 -> 237.6 mm
- net DIF0: track 234.5 -> 233.5 mm
- net N$30: track 40.4 -> 39.4 mm
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
Commit message: Maybe done?
Parts:
- moved C5B 1.50 mm to (84.1, 119.1)
- moved C3B 0.75 mm to (88.8, 124.2)
- moved C14O 0.35 mm to (93.0, 76.8)
- moved C12O 0.35 mm to (102.5, 82.9)
Routing:
- net MCLK: track 131.1 -> 175.5 mm
- net N$117: track 27.8 -> 32.5 mm
- net N$92: track 27.9 -> 32.1 mm
- net +5V/4: track 58.0 -> 56.5 mm
- net AGND: track 21.0 -> 19.5 mm
- net +5V/2: track 94.1 -> 94.8 mm
Other:
- board text removed: "AOLP DGND AOLN AORN DGND AORP"
