File: AK4493-Combi3.brd (EAGLE design)
At the start: 178 x 151.3 mm, 222 parts, among them IC1 LT3042, IC3 AK4493, IC4 LT3042, IC4A SN74ABT273DBR, IC5 LT3042, IC6 LT3042, IC7 LT3042, IC8 LT3042, IC9 AK4493, J15 XR2A-0811-N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

Commit message: More slight changes
Routing:
- net AGND: track 19.5 -> 23.7 mm
- net DGND: track 2.14 -> 0.00 mm, vias 105 -> 107
