File: AK4493-Combi4.sch (EAGLE design)
At the start: 226 parts, among them IC1 LT3042, IC3 AK4493, IC4 LT3042, IC4A SN74ABT273DBR, IC5 LT3042, IC6 LT3042, IC7 LT3042, IC8 LT3042, IC9 AK4493, J15 XR2A-0811-N, J16 XR2A-0811-N, J17 XR2A-0811-N, J18 XR2A-0811-N, J19 XR2A-0811-N, J20 XR2A-0811-N, J26 SJ-63033A, J27 1935161, U1 AZ1117H-5.0TRE1, X1 JST-XH-07-PIN-ROUND-PAD, X4 JST-XH-04-PIN-ROUND-PAD

Commit message: Progress
Parts:
- removed C6P1, C7P1: 68u, Dual Mono Amp Library:500HXW68MEFR14.5X45
- added C10P, C8P, C9P: 68u, Dual Mono Amp Library:500HXW68MEFR14.5X45
- C1P1, C2P1, C3P1, C5P1: device Dual Mono Amp Library:500HXW68MEFR14.5X45 -> Dual Mono Amp Library:35PX6800MEFC18X35.5
Connections:
- removed net VCC/1: C1P1.+, C2.1, C20A.1, C20B.1, C20C.1, C20D.1, C20E.1, C20F.1, C21A.1, C21B.1, C21C.1, C21D.1, C21E.1, C21F.1, C2P1.+, C3P1.+, C4.1, C5P1.+, C6P1.+, C7P1.+, D7.K, D8.K, IC1.EN/UV, IC1.IN, IC4.EN/UV, IC4.IN, IC5.EN/UV, IC5.IN, IC6.EN/UV, IC6.IN, IC7.EN/UV, IC7.IN, IC8.EN/UV, IC8.IN, J15.7, J15.8, J16.7, J16.8, J17.7, J17.8, J18.7, J18.8, J19.7, J19.8, J20.7, J20.8, R8A.1, R8B.1, R8C.1, R8D.1, R8E.1, R8F.1, U1.INPUT
- net +240VDC: now also C10P.+, C8P.+, C9P.+, R4P.2
- net 115_VAC_BLK: now also IN.7; no longer IN.4
- net 115_VAC_RED: now also IN.6; no longer IN.3
- net 6.3_VAC_BLU: now also IN.2; no longer IN.5
- net 6.3_VAC_GRN: now also IN.3; no longer IN.6
- net 66.3VAC/1: now also IN.5; no longer IN.1
- net 66.3VAC/2: now also IN.4; no longer IN.2
- net DGND: now also C10P.-, C8P.-, C9P.-; no longer C6P1.-, C7P1.-
- net PE: now also IN.1; no longer IN.7
- net VCC: now also C1P1.+, C2.1, C20A.1, C20B.1, C20C.1, C20D.1, C20E.1, C20F.1, C21A.1, C21B.1, C21C.1, C21D.1, C21E.1, C21F.1, C2P1.+, C3P1.+, C4.1, C5P1.+, D7.K, D8.K, IC1.EN/UV, IC1.IN, IC4.EN/UV, IC4.IN, IC5.EN/UV, IC5.IN, IC6.EN/UV, IC6.IN, IC7.EN/UV, IC7.IN, IC8.EN/UV, IC8.IN, J15.7, J15.8, J16.7, J16.8, J17.7, J17.8, J18.7, J18.8, J19.7, J19.8, J20.7, J20.8, R8A.1, R8B.1, R8C.1, R8D.1, R8E.1, R8F.1, U1.INPUT; no longer R4P.2
Other:
- moved on the sheet: IN
