File: AK4493-Combi5.brd (EAGLE design)
At the start: 177.8 x 151.3 mm, 227 parts, among them IC1 LT3042, IC3 AK4493, IC4 LT3042, IC4A SN74ABT273DBR, IC5 LT3042, IC6 LT3042, IC7 LT3042, IC8 LT3042, IC9 AK4493, J15 XR2A-0811-N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

Commit message: Progress
Connections:
- removed net N$138: DIF2.3, IC3.14, IC3.15, IC3.17, J1.5
- net +3V3: now also DIF2.3, IC3.14, IC3.15, IC3.17, J1.5
- net DGND: now also IC3.18, IC9.18
Routing:
- net +3V3: track 173.5 -> 178.7 mm
- net DGND: track 8.58 -> 13.6 mm
- net N$138: track 4.48 -> 0.00 mm
- removed copper zone on layer 16, net N$138
