File: AK4493-Combi6.sch (EAGLE design)
At the start: 227 parts, among them IC1 LT3042, IC3 AK4493, IC4 LT3042, IC4A SN74ABT273DBR, IC5 LT3042, IC6 LT3042, IC7 LT3042, IC8 LT3042, IC9 AK4493, J15 XR2A-0811-N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

Commit message: Progress
Parts:
- added C17O, C19O: 0.1uF, 35V, Dual Mono Amp Library:MKS4B031002A00JC00
Connections:
- new net N$35: C19O.2, R1O.1
- new net N$48: C17O.2, R13O.1
- new net N$56: IC3.DIF1, J1.6
- new net N$58: IC3.DIF0, J1.7
- net DIF0: no longer IC3.DIF0, J1.7
- net DIF1: no longer IC3.DIF1, J1.6
- net L+: now also C19O.1; no longer R1O.1
- net R+: now also C17O.1; no longer R13O.1
