File: DAC_GainOutputStage4.brd (EAGLE design)
At the start: 110 x 102.8 mm, 68 parts, among them J1 1935190, J3 SJ-63033A, U1 LM317MQDCYR, U2 LM317MQDCYR

Commit message: Progress
Routing:
- net N$5: track 68.1 -> 65.2 mm
