File: DAC_GainOutputStage6.brd (EAGLE design)
At the start: 110 x 105.3 mm, 70 parts, among them J1 1935190, J3 SJ-63033A, U1 LM317MQDCYR, U2 LM317MQDCYR

Commit message: Finished updated design
Parts:
- moved U1 1.55 mm to (4.67, 44.0)
- moved U2 1.55 mm to (105.3, 44.0)
- turned R17 to 90 degrees
- turned R18 to 270 degrees
Routing:
- net N$22: track 0.00 -> 102.9 mm
- net N$7: track 0.00 -> 91.3 mm
- net N$5: track 0.00 -> 75.8 mm
- net N$26: track 0.00 -> 64.2 mm
- net N$13: track 0.00 -> 58.7 mm, vias 0 -> 1
- net N$17: track 0.00 -> 56.1 mm
- net N$16: track 0.00 -> 55.4 mm
- net N$27: track 0.00 -> 54.6 mm
- net N$29: track 0.00 -> 52.6 mm
- net N$3: track 6.65 -> 58.8 mm
- net N$23: track 18.7 -> 67.8 mm
- net N$2: track 0.00 -> 43.5 mm
- net N$14: track 0.00 -> 42.0 mm
- net N$6: track 0.00 -> 41.3 mm
- net N$4: track 0.00 -> 37.9 mm
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