File: DAC_GainOutputStage8.brd (EAGLE design)
At the start: 112 x 110.3 mm, 78 parts, among them J1 1935190, J3 SJ-63033A, U1 LM317MTG, U2 LM317MTG

Commit message: Progress
Parts:
- removed C5, C6: DCP4G056007GD4KSSD, DCP4G056007GD4KSSD:DCP4G056007GD4KSSD
- C21O, C21O1: device Dual Mono Amp Library:DCP4G053006ID2KSSD -> Dual Mono Amp Library:DCP4G056007GD4KSSD
- moved R9 44.9 mm to (36.1, 30.4), turned to 180 degrees
- moved R15 43.3 mm to (75.9, 30.4), turned to 0 degrees
- moved D3 37.1 mm to (22.1, 30.4), turned to 180 degrees
- moved D6 36.2 mm to (89.9, 30.4), turned to 0 degrees
- moved Z1 28.4 mm to (14.5, 25.5)
- moved Z2 28.4 mm to (41.1, 25.5)
- moved Z5 28.4 mm to (70.8, 25.5)
- moved Z6 28.4 mm to (97.5, 25.5)
- moved D1 13.0 mm to (43.8, 76.9)
- moved D4 13.0 mm to (68.1, 76.9)
- moved R13 13.0 mm to (95.5, 68.7)
- moved R19 13.0 mm to (32.4, 68.7)
- moved R2 13.0 mm to (7.00, 71.9)
- moved R20 13.0 mm to (79.6, 68.7)
- moved R3O 13.0 mm to (2.03, 71.9)
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Connections:
- net L_OUT: now also C21O1.4
- net N$18: now also C21O.3
- net N$3: now also C21O1.3
- net R_OUT: now also C21O.4
Routing:
- net N$29: track 66.2 -> 46.8 mm
- net N$26: track 71.5 -> 58.2 mm
- net R_OUT: track 39.8 -> 50.1 mm
- net L_OUT: track 35.3 -> 45.1 mm
- net N$18: track 57.0 -> 66.2 mm
- net N$3: track 66.0 -> 74.1 mm
- net N$23: track 68.9 -> 60.9 mm
- net N$27: track 62.3 -> 57.2 mm
- net +240VDC: track 279.9 -> 281.1 mm
Other:
- board size 112 x 110.3 mm -> 112 x 118.3 mm
