File: DAC_GainOutputStage8.sch (EAGLE design)
At the start: 78 parts, among them J1 1935190, J3 SJ-63033A, U1 LM317MTG, U2 LM317MTG

Commit message: Progress
Parts:
- removed C5, C6: DCP4G056007GD4KSSD, DCP4G056007GD4KSSD:DCP4G056007GD4KSSD
- C21O, C21O1: device Dual Mono Amp Library:DCP4G053006ID2KSSD -> Dual Mono Amp Library:DCP4G056007GD4KSSD
Changed lines of the file:
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@@
 <part name="SX1" library="Dual Mono Amp Library" library_urn="urn:adsk.wipprod:fs.file:vf.VjdQUjkvQKmMNRW9J90YWw" deviceset="VT9" device="-PT" package3d_urn="urn:adsk.eagle:package:4683/1"/>
 <part name="U$8" library="Dual Mono Amp Library" library_urn="urn:adsk.wipprod:fs.file:vf.VjdQUjkvQKmMNRW9J90YWw" deviceset="+240VDC" device=""/>
-<part name="C21O" library="Dual Mono Amp Library" library_urn="urn:adsk.wipprod:fs.file:vf.VjdQUjkvQKmMNRW9J90YWw" deviceset="DCP4G053006ID2KSSD" device="" value="30uF/400V"/>
+<part name="C21O" library="Dual Mono Amp Library" library_urn="urn:adsk.eagle:library:47621477" deviceset="DCP4G056007GD4KSSD" device="" package3d_urn="urn:adsk.eagle:package:50745978/1" value="30uF/400V"/>
 <part name="AGND3" library="Dual Mono Amp Library" library_urn="urn:adsk.wipprod:fs.file:vf.VjdQUjkvQKmMNRW9J90YWw" deviceset="AGND" device=""/>
 <part name="U$9" library="Dual Mono Amp Library" library_urn="urn:adsk.wipprod:fs.file:vf.VjdQUjkvQKmMNRW9J90YWw" deviceset="66.3VAC/1" device=""/>
@@
 <part name="SX2" library="Dual Mono Amp Library" library_urn="urn:adsk.wipprod:fs.file:vf.VjdQUjkvQKmMNRW9J90YWw" deviceset="VT9" device="-PT" package3d_urn="urn:adsk.eagle:package:4683/1"/>
 <part name="U$3" library="Dual Mono Amp Library" library_urn="urn:adsk.wipprod:fs.file:vf.VjdQUjkvQKmMNRW9J90YWw" deviceset="+240VDC" device=""/>
-<part name="C21O1" library="Dual Mono Amp Library" library_urn="urn:adsk.wipprod:fs.file:vf.VjdQUjkvQKmMNRW9J90YWw" deviceset="DCP4G053006ID2KSSD" device="" value="30uF/400V"/>
+<part name="C21O1" library="Dual Mono Amp Library" library_urn="urn:adsk.eagle:library:47621477" deviceset="DCP4G056007GD4KSSD" device="" package3d_urn="urn:adsk.eagle:package:50745978/1" value="30uF/400V"/>
 <part name="AGND1" library="Dual Mono Amp Library" library_urn="urn:adsk.wipprod:fs.file:vf.VjdQUjkvQKmMNRW9J90YWw" deviceset="AGND" device=""/>
 <part name="U$4" library="Dual Mono Amp Library" library_urn="urn:adsk.wipprod:fs.file:vf.VjdQUjkvQKmMNRW9J90YWw" deviceset="66.3VAC/1" device=""/>
@@
 <part name="R19" library="Dual Mono Amp Library" library_urn="urn:adsk.eagle:library:47621477" deviceset="CPF215K000FKE14" device="" package3d_urn="urn:adsk.eagle:package:23568/2" value="15k"/>
 <part name="R20" library="Dual Mono Amp Library" library_urn="urn:adsk.eagle:library:47621477" deviceset="CPF215K000FKE14" device="" package3d_urn="urn:adsk.eagle:package:23568/2" value="15k"/>
-<part name="C5" library="DCP4G056007GD4KSSD" deviceset="DCP4G056007GD4KSSD" device=""/>
-<part name="C6" library="DCP4G056007GD4KSSD" deviceset="DCP4G056007GD4KSSD" device=""/>
 </parts>
 <sheets>
@@
 <attribute name="VALUE" x="158.75" y="171.958" size="1.778" layer="96"/>
 </instance>
-<instance part="C5" gate="G$1" x="60.96" y="81.28" smashed="yes">
-<attribute name="NAME" x="77.47" y="88.9" size="1.778" layer="95" align="center-left"/>
-<attribute name="VALUE" x="77.47" y="86.36" size="1.778" layer="96" align="center-left"/>
-</instance>
-<instance part="C6" gate="G$1" x="111.76" y="81.28" smashed="yes">
-<attribute name="NAME" x="128.27" y="88.9" size="1.778" layer="95" align="center-left"/>
-<attribute name="VALUE" x="128.27" y="86.36" size="1.778" layer="96" align="center-left"/>
-</instance>
 </instances>
