File: AK4493-Combi8.brd (EAGLE design)
At the start: 112 x 118.3 mm, 111 parts, among them J1 1935239, J3 SJ-63033A, J4 1935239, U1 LM317MTG, U2 LM317MTG

Commit message: Moar combi progress
Parts:
- removed SH1, SH2: SHORTA5, Dual Mono Amp Library:SHORT_ALL-50
Connections:
- removed net DGND: C4P.2, R5P.1
- net AGND/1: no longer SH2.1
- net AGND/2: no longer SH1.1
- net DGND/1: no longer SH2.2
- net DGND/2: now also C4P.2, R5P.1; no longer SH1.2
Routing:
- added copper zone on layer 1, net DGND/2
- removed copper zone on layer 1, net DGND

Commit message: Progress
Parts:
- added SH1, SH2: SHORTA5, Dual Mono Amp Library:SHORT_ALL-50
Connections:
- net AGND/1: now also SH1.2
- net AGND/2: now also SH2.2
- net DGND/1: now also SH1.1
- net DGND/2: now also SH2.1
Routing:
- net 115_VAC_RED/2: track 8.90 -> 73.0 mm
- net N$44: track 17.8 -> 40.5 mm
- net 115_VAC_BLK/2: track 18.7 -> 38.2 mm
- net 66.3VAC/BRN/2: track 175.1 -> 193.7 mm
- net 66.3VAC/ORG/2: track 217.7 -> 203.2 mm
- net N$43: track 25.6 -> 31.4 mm
- added copper zone on layer 1, net AGND/1

Commit message: Progress
Parts:
- removed C4P1: UCY2E220MPD1TD, UCY2E220MPD1TD:CAPPRD500W60D1025H1750
- removed R2P1, R3P1: 220, rcl:0411/15
- removed R4P1: 300k, rcl:0411/15
- removed R5P1: 100k, rcl:0411/15
- removed SH1: SHORTA5, Dual Mono Amp Library:SHORT_ALL-50
- added C18A, C18B, C18D: 4.7u, Dual Mono Amp Library:CAPC2013X140N
- added C19A, C19B, C19D: 22u, Dual Mono Amp Library:C1206
- added C20A, C20B, C20D: 10u, Dual Mono Amp Library:CAPC2012X135N
- added C21A, C21B, C21D: 0.1u, Dual Mono Amp Library:CAPC2012X135N
- added C26A, C27A: 4.7u, Ceramic Capacitor X7R, Dual Mono Amp Library:CAPC2013X140N
- added C28A: 0.1u, Ceramic Capacitor X7R, Dual Mono Amp Library:CAPC2012X135N
- added IC1, IC2, IC5: LT3042, Dual Mono Amp Library:SOP50P490X110-11N
- added IC3: LM317MQDCYR, Dual Mono Amp Library:SOT230P700X180-4N
- added J17, J5: XR2A-0811-N, XR2A-0811-N:DIPS762W51P254L1016H390Q8N
- added LDO7: LP5907-1.8V, Dual Mono Amp Library:SOT95P280X145-5N
- added R6A, R6B, R6D: 1k, Dual Mono Amp Library:RESC2012X60N
- added R7A, R7B, R7D: 33k, Dual Mono Amp Library:R0805
- added R8A, R8B, R8D: 200k, Dual Mono Amp Library:R0805
- J1: value 1935239 -> XR2A-0811-N; device Dual Mono Amp Library:1935239 -> XR2A-0811-N:DIPS762W51P254L1016H390Q8N
- moved J1 269.7 mm to (123.3, 144.8), flipped to the bottom, turned to 270 degrees
- moved D11 113.2 mm to (-50.0, -184.0)
- moved D13 107.1 mm to (-50.0, -188.0)
- moved D12 103.2 mm to (-29.0, -184.0)
- moved D14 103.2 mm to (-29.0, -188.0)
- moved C1P1 101.0 mm to (-51.0, -121.0)
- moved C2P1 101.0 mm to (-35.0, -121.0)
- moved C3P1 101.0 mm to (-19.0, -121.0)
- moved C5P1 101.0 mm to (-51.0, -137.0)
- moved C6P1 101.0 mm to (-35.0, -137.0)
- moved C7P1 101.0 mm to (-19.0, -137.0)
- moved R6P1 101.0 mm to (-30.0, -180.0)
- moved C1P 5.31 mm to (100.3, 21.2)
- moved C5P 5.31 mm to (100.3, 59.1)
- moved C6P 5.31 mm to (100.3, 42.4)
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Connections:
- removed net 115_VAC_BLK/1: D11.1, D14.2, J1.2
- removed net 115_VAC_RED/1: D12.1, D13.2, J1.3
- removed net 6.3_VAC_BLU/1: J1.8
- removed net 6.3_VAC_GRN/1: J1.9
- removed net DGND/1: C1P1.2, C2P1.2, C3P1.2, C4P1.2, C5P1.2, C6P1.2, C7P1.2, D11.2, D12.2, R5P1.1, SH1.1
- new net +3V3: C18A.1, C26A.1, IC2.10, IC2.9, J5.6, LDO7.1, LDO7.3
- new net +5V/1: C18D.1, IC1.10, IC1.9, J1.6
- new net +5V/2: C18B.1, IC5.10, IC5.9, J17.6
- new net DGND: C26A.2, C27A.2, C28A.2, LDO7.2, LDO7.DGND, LDO7.DGND2, LDO7.DGND3
- new net N$103: C19B.1, IC5.7, J17.4, R7B.1
- new net N$49: IC1.4, J1.1, R8D.2
- new net N$50: IC1.5, J1.2, R6D.1
- new net N$51: IC1.6, J1.3
- new net N$52: C19D.1, IC1.7, J1.4, R7D.1
- new net N$53: IC2.4, J5.1, R8A.2
- new net N$54: IC2.5, J5.2, R6A.1
- new net N$55: IC2.6, J5.3
- new net N$56: C19A.1, IC2.7, J5.4, R7A.1
- new net N$57: C1P1.1, D13.1, D14.1
- new net N$58: C2P1.1, R6P1.2
- new net N$65: C27A.1, C28A.1, LDO7.5
- new net VCC/2: C20A.1, C20B.1, C20D.1, C21A.1, C21B.1, C21D.1, C3P1.1, C5P1.1, C6P1.1, C7P1.1, IC1.1, IC1.2, IC1.3, IC2.1, IC2.2, IC2.3, IC5.1, IC5.2, IC5.3, J1.7, J1.8, J17.7, J17.8, J5.7, J5.8, R6P1.1, R8A.1, R8B.1, R8D.1
- net +240VDC/1: no longer C3P1.1, C5P1.1, C6P1.1, C7P1.1, R4P1.2, R6P1.1
- net 6.3_VAC_BLU/2: now also D11.1, D14.2
- net 6.3_VAC_GRN/2: now also D12.1, D13.2
- net 66.3VAC/BRN/1: no longer J1.7, R3P1.1
- net 66.3VAC/ORG/1: no longer J1.6, R2P1.2
- net AGND/1: no longer SH1.2
- net AGND/2: now also C1P.2, C2P.2, C3P.2, C4P.2, C5P.2, C6P.2, C7P.2, D7.2, D8.2, R5P.1
- net DGND/2: now also C18A.2, C18B.2, C18D.2, C19A.2, C19A.DGND, C19B.2, C19B.DGND, C19D.2, C19D.DGND, C1P1.2, C20A.2, C20B.2, C20D.2, C21A.2, C21B.2, C21D.2, C2P1.2, C3P1.2, C5P1.2, C6P1.2, C7P1.2, D11.2, D12.2, IC1.11, IC1.8, IC1.P$1, IC1.P$2, IC1.P$3, IC1.P$4, IC1.P$5, IC1.P$6, IC2.11, IC2.8, IC2.P$1, IC2.P$2, IC2.P$3, IC2.P$4, IC2.P$5, IC2.P$6, IC5.11, IC5.8, IC5.P$1, IC5.P$2, IC5.P$3, IC5.P$4, IC5.P$5, IC5.P$6, J1.5, J17.5, J5.5, R6A.2, R6B.2, R6D.2, R7A.2, R7B.2, R7D.2; no longer C1P.2, C2P.2, C3P.2, C4P.2, C5P.2, C6P.2, C7P.2, D7.2, D8.2, R5P.1
- net N$46: now also IC5.4, J17.1, R8B.2; no longer C1P1.1, D13.1, D14.1, J1.4
- net N$47: now also IC5.5, J17.2, R6B.1; no longer C2P1.1, J1.5, R6P1.2
- net N$48: now also IC5.6, J17.3; no longer C4P1.1, R2P1.1, R3P1.2, R4P1.1, R5P1.2
- net PE: no longer J1.1
Routing:
- net VCC/2: track 0.00 -> 45.1 mm
- net N$52: track 0.00 -> 10.9 mm
- net N$103: track 0.00 -> 10.9 mm
- net N$56: track 0.00 -> 10.9 mm
- net +3V3: track 0.00 -> 9.61 mm
- net +5V/2: track 0.00 -> 9.61 mm
- net +5V/1: track 0.00 -> 9.61 mm
- net N$49: track 0.00 -> 7.84 mm
- net N$46: track 0.00 -> 7.84 mm
- net N$53: track 0.00 -> 7.84 mm
- net N$54: track 0.00 -> 6.08 mm
- net N$50: track 0.00 -> 6.08 mm
- net N$47: track 0.00 -> 6.08 mm
- net 66.3VAC/ORG/2: track 203.2 -> 198.2 mm
- net N$48: track 0.00 -> 3.20 mm
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- added copper zone on layer 16, net +5V/1
- added copper zone on layer 16, net +5V/2
- added copper zone on layer 16, net +5V/3
- added copper zone on layer 16, net DGND/2
- added copper zone on layer 16, net VCC/2
- removed copper zone on layer 16, net AGND/2
