File: AK4493-Combi8.sch (EAGLE design)
At the start: 111 parts, among them J1 1935161, J3 SJ-63033A, J4 1935161, U1 LM317MTG, U2 LM317MTG

Commit message: Moar combi progress
Parts:
- removed IN, IN1: 1935213, 1935213:1935213
- J1, J4: value 1935161 -> 1935239; device 1935161:1935161 -> Dual Mono Amp Library:1935239
Connections:
- removed net 115_VAC_BLK: D10.A, D11.K, D14.A, D7.K, IN.4, IN1.4
- removed net 115_VAC_RED: D12.K, D13.A, D8.K, D9.A, IN.3, IN1.3
- removed net 6.3_VAC_BLU: IN.7, IN1.7
- removed net 6.3_VAC_GRN: IN.6, IN1.6
- removed net AGND: C1.2, C2.2, C3.2, C4.2, J13.2, J13.5, J2.2, J2.5, J3.SLEEVE, R10.1, R11O.2, R15.1, R16.1, R19O.1, R20O.2, R20O1.1, R20O2.1, R21O.1, R22O.2, R28O.1, R29O.2, R30O.1, R3O.2, R3O1.2, R9.1, U1.ADJ, U2.ADJ, Z1.C, Z6.C
- removed net DGND: C1P.-, C1P1.-, C2P.-, C2P1.-, C3P.-, C3P1.-, C4P.-, C4P1.-, C5P.-, C5P1.-, C6P.-, C6P1.-, C7P.-, C7P1.-, D11.A, D12.A, D7.A, D8.A, R5P.1, R5P1.1
- new net +240VDC/1: C1.1, C3.1, C3P1.+, C5P1.+, C6P1.+, C7P1.+, R17.1, R19.2, R4P1.2, R5.2, R6P1.1
- new net 115_VAC_BLK/1: D11.K, D14.A, J1.2
- new net 115_VAC_BLK/2: D10.A, D7.K, J4.2
- new net 115_VAC_RED/1: D12.K, D13.A, J1.3
- new net 115_VAC_RED/2: D8.K, D9.A, J4.3
- new net 6.3_VAC_BLU/1: J1.8
- new net 6.3_VAC_BLU/2: J4.8
- new net 6.3_VAC_GRN/1: J1.9
- new net 6.3_VAC_GRN/2: J4.9
- new net 66.3VAC/BRN/1: J1.7, R3P1.1, SX1.4, SX3.4
- new net 66.3VAC/ORG/1: J1.6, R2P1.2, SX1.5, SX3.5
- new net AGND/1: C1.2, C3.2, J13.2, J13.5, J3.SLEEVE, R10.1, R11O.2, R19O.1, R20O.2, R20O1.1, R21O.1, R3O.2, R9.1, U1.ADJ, Z1.C
- new net AGND/2: C2.2, C4.2, J2.2, J2.5, R15.1, R16.1, R20O2.1, R22O.2, R28O.1, R29O.2, R30O.1, R3O1.2, U2.ADJ, Z6.C
- new net DGND/1: C1P1.-, C2P1.-, C3P1.-, C4P1.-, C5P1.-, C6P1.-, C7P1.-, D11.A, D12.A, R5P1.1
- new net DGND/2: C1P.-, C2P.-, C3P.-, C4P.-, C5P.-, C6P.-, C7P.-, D7.A, D8.A, R5P.1
- net +240VDC/2: no longer C1.1, C3.1, C3P1.+, C5P1.+, C6P1.+, C7P1.+, R17.1, R19.2, R4P1.2, R5.2, R6P1.1
- net 66.3VAC/BRN/2: now also J4.7; no longer IN.1, IN1.1, R3P1.1, SX1.4, SX3.4
- net 66.3VAC/ORG/2: now also J4.6; no longer IN.2, IN1.2, R2P1.2, SX1.5, SX3.5
- net N$43: now also J4.4; no longer J4.1
- net N$44: now also J4.5; no longer J4.2
- net N$46: now also J1.4; no longer J1.1
- net N$47: now also J1.5; no longer J1.2
- net PE: now also J1.1, J4.1; no longer IN.5, IN1.5
Other:
- moved on the sheet: C1, C11O, C12O, C13O, C14O, C15O, C1P, C1P1, C2, C21O, C21O1, C24O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

Commit message: Progress
Parts:
- added SH1, SH2: SHORTA5, Dual Mono Amp Library:SHORTA5
Connections:
- net AGND/1: now also SH1.P$2
- net AGND/2: now also SH2.P$2
- net DGND/1: now also SH1.P$1
- net DGND/2: now also SH2.P$1
Changed lines of the file:
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@@
 <part name="U$20" library="Dual Mono Amp Library" library_urn="urn:adsk.eagle:library:47621477" deviceset="66.3VAC/ORG/1" device=""/>
 <part name="J1" library="Dual Mono Amp Library" library_urn="urn:adsk.eagle:library:47621477" deviceset="1935239" device="" package3d_urn="urn:adsk.eagle:package:50748024/1"/>
+<part name="SH1" library="Dual Mono Amp Library" library_urn="urn:adsk.eagle:library:47621477" deviceset="SHORT" device="A5" package3d_urn="urn:adsk.eagle:package:47621621/1"/>
+<part name="SH2" library="Dual Mono Amp Library" library_urn="urn:adsk.eagle:library:47621477" deviceset="SHORT" device="A5" package3d_urn="urn:adsk.eagle:package:47621621/1"/>
+<part name="SUPPLY5" library="Dual Mono Amp Library" library_urn="urn:adsk.eagle:library:47621477" deviceset="DGND/1" device=""/>
+<part name="AGND2" library="Dual Mono Amp Library" library_urn="urn:adsk.eagle:library:47621477" deviceset="AGND/1" device=""/>
+<part name="AGND20" library="Dual Mono Amp Library" library_urn="urn:adsk.eagle:library:47621477" deviceset="AGND/2" device=""/>
+<part name="SUPPLY6" library="Dual Mono Amp Library" library_urn="urn:adsk.eagle:library:47621477" deviceset="DGND/2" device=""/>
 </parts>
 <sheets>
@@
 <attribute name="NAME" x="-165.1" y="219.71" size="1.778" layer="95" rot="MR90" align="center-left"/>
 <attribute name="VALUE" x="-167.64" y="219.71" size="1.778" layer="96" rot="MR90" align="center-left"/>
+</instance>
+<instance part="SH1" gate="G$1" x="-157.48" y="73.66" smashed="yes" rot="R90">
+<attribute name="NAME" x="-158.75" y="71.4375" size="1.778" layer="95" rot="R90"/>
+</instance>
+<instance part="SH2" gate="G$1" x="157.48" y="73.66" smashed="yes" rot="R90">
+<attribute name="NAME" x="156.21" y="71.4375" size="1.778" layer="95" rot="R90"/>
+</instance>
+<instance part="SUPPLY5" gate="G$1" x="-157.48" y="66.04" smashed="yes" rot="MR0">
+<attribute name="VALUE" x="-154.813" y="62.865" size="1.778" layer="96" rot="MR0"/>
+</instance>
+<instance part="AGND2" gate="G$1" x="-157.48" y="81.28" smashed="yes" rot="MR180">
+<attribute name="VALUE" x="-165.1" y="86.36" size="1.778" layer="96" rot="MR270"/>
+</instance>
+<instance part="AGND20" gate="G$1" x="157.48" y="81.28" smashed="yes" rot="R180">
+<attribute name="VALUE" x="160.02" y="86.36" size="1.778" layer="96" rot="R270"/>
+</instance>
+<instance part="SUPPLY6" gate="G$1" x="157.48" y="66.04" smashed="yes">
+<attribute name="VALUE" x="154.813" y="62.865" size="1.778" layer="96"/>
 </instance>
 </instances>
@@
 <wire x1="-58.42" y1="78.74" x2="-58.42" y2="66.04" width="0.1524" layer="91"/>
 </segment>
+<segment>
+<pinref part="SH1" gate="G$1" pin="P$2"/>
+<pinref part="AGND2" gate="G$1" pin="AGND/1"/>
+<wire x1="-157.48" y1="78.74" x2="-157.48" y2="76.2" width="0.1524" layer="91"/>
+</segment>
 </net>
 <net name="AGND/2" class="0">
@@
 <wire x1="35.56" y1="170.18" x2="35.56" y2="172.72" width="0.1524" layer="91"/>
 <junction x="35.56" y="172.72"/>
+</segment>
+<segment>
+<pinref part="SH2" gate="G$1" pin="P$2"/>
+<pinref part="AGND20" gate="G$1" pin="AGND/2"/>
+<wire x1="157.48" y1="78.74" x2="157.48" y2="76.2" width="0.1524" layer="91"/>
 </segment>
 </net>
@@
 <junction x="182.88" y="60.96"/>
 </segment>
+<segment>
+<pinref part="SH2" gate="G$1" pin="P$1"/>
+<pinref part="SUPPLY6" gate="G$1" pin="DGND/2"/>
+<wire x1="157.48" y1="68.58" x2="157.48" y2="71.12" width="0.1524" layer="91"/>
+</segment>
 </net>
 <net name="66.3VAC/BRN/1" class="0">
@@
 <junction x="-134.62" y="152.4"/>
 </segment>
-</net>
+<segment>
+<pinref part="SH1" gate="G$1" pin="P$1"/>
+<pinref part="SUPPLY5" gate="G$1" pin="DGND/1"/>
+<wire x1="-157.48" y1="68.58" x2="-157.48" y2="71.12" width="0.1524" layer="91"/>
+</segment>
+</net>

Commit message: Progress
Parts:
- removed C4P1: UCY2E220MPD1TD, UCY2E220MPD1TD:UCY2E220MPD1TD
- removed R2P1, R3P1: 220, rcl:R-US_0411/15
- removed R4P1: 300k, rcl:R-US_0411/15
- removed R5P1: 100k, rcl:R-US_0411/15
- removed SH1: SHORTA5, Dual Mono Amp Library:SHORTA5
- added C18A, C18B, C18D: 4.7u, Dual Mono Amp Library:EMK212ABJ475KG-T
- added C19A, C19B, C19D: 22u, Dual Mono Amp Library:EMK316BB7226ML-T
- added C20A, C20B, C20D: 10u, Dual Mono Amp Library:EMK212BB7106KG-T
- added C21A, C21B, C21D: 0.1u, Dual Mono Amp Library:EMF212B7104KGHT
- added C26A, C27A: 4.7u, Ceramic Capacitor X7R, Dual Mono Amp Library:EMK212ABJ475KG-T
- added C28A: 0.1u, Ceramic Capacitor X7R, Dual Mono Amp Library:EMF212B7104KGHT
- added IC1, IC2, IC5: LT3042, Dual Mono Amp Library:LT3042
- added IC3: LM317MQDCYR, Dual Mono Amp Library:LM317MQDCYR
- added J17, J5: XR2A-0811-N, XR2A-0811-N:XR2A-0811-N
- added LDO7: LP5907-1.8V, Dual Mono Amp Library:LP5907-1.8V
- added R6A, R6B, R6D: 1k, Dual Mono Amp Library:CHP0805-FX-1001ELF
- added R7A, R7B, R7D: 33k, Dual Mono Amp Library:CPF0805B51KE1
- added R8A, R8B, R8D: 200k, Dual Mono Amp Library:RR1220P-204-D
- J1: value 1935239 -> XR2A-0811-N; device Dual Mono Amp Library:1935239 -> XR2A-0811-N:XR2A-0811-N
Connections:
- removed net 115_VAC_BLK/1: D11.K, D14.A, J1.2
- removed net 115_VAC_RED/1: D12.K, D13.A, J1.3
- removed net 6.3_VAC_BLU/1: J1.8
- removed net 6.3_VAC_GRN/1: J1.9
- removed net DGND/1: C1P1.-, C2P1.-, C3P1.-, C4P1.-, C5P1.-, C6P1.-, C7P1.-, D11.A, D12.A, R5P1.1, SH1.P$1
- new net +3V3: C18A.1, C26A.1, IC2.OUT, IC2.OUTS, J5.6, LDO7.EN, LDO7.VIN
- new net +5V/1: C18D.1, IC1.OUT, IC1.OUTS, J1.6
- new net +5V/2: C18B.1, IC5.OUT, IC5.OUTS, J17.6
- new net DGND: C26A.2, C27A.2, C28A.2, LDO7.GND
- new net N$103: C19B.1, IC5.SET, J17.4, R7B.1
- new net N$49: IC1.PG, J1.1, R8D.2
- new net N$50: IC1.ILIM, J1.2, R6D.1
- new net N$51: IC1.PGFB, J1.3
- new net N$52: C19D.1, IC1.SET, J1.4, R7D.1
- new net N$53: IC2.PG, J5.1, R8A.2
- new net N$54: IC2.ILIM, J5.2, R6A.1
- new net N$55: IC2.PGFB, J5.3
- new net N$56: C19A.1, IC2.SET, J5.4, R7A.1
- new net N$57: C1P1.+, D13.K, D14.K
- new net N$58: C2P1.+, R6P1.2
- new net N$65: C27A.1, C28A.1, LDO7.VOUT
- new net VCC/2: C20A.1, C20B.1, C20D.1, C21A.1, C21B.1, C21D.1, C3P1.+, C5P1.+, C6P1.+, C7P1.+, IC1.EN/UV, IC1.IN, IC2.EN/UV, IC2.IN, IC5.EN/UV, IC5.IN, J1.7, J1.8, J17.7, J17.8, J5.7, J5.8, R6P1.1, R8A.1, R8B.1, R8D.1
- net +240VDC/1: no longer C3P1.+, C5P1.+, C6P1.+, C7P1.+, R4P1.2, R6P1.1
- net 6.3_VAC_BLU/2: now also D11.K, D14.A
- net 6.3_VAC_GRN/2: now also D12.K, D13.A
- net 66.3VAC/BRN/1: no longer J1.7, R3P1.1
- net 66.3VAC/ORG/1: no longer J1.6, R2P1.2
- net AGND/1: no longer SH1.P$2
- net AGND/2: now also C1P.-, C2P.-, C3P.-, C4P.-, C5P.-, C6P.-, C7P.-, D7.A, D8.A, R5P.1
- net DGND/2: now also C18A.2, C18B.2, C18D.2, C19A.2, C19B.2, C19D.2, C1P1.-, C20A.2, C20B.2, C20D.2, C21A.2, C21B.2, C21D.2, C2P1.-, C3P1.-, C5P1.-, C6P1.-, C7P1.-, D11.A, D12.A, IC1.GND, IC2.GND, IC5.GND, J1.5, J17.5, J5.5, R6A.2, R6B.2, R6D.2, R7A.2, R7B.2, R7D.2; no longer C1P.-, C2P.-, C3P.-, C4P.-, C5P.-, C6P.-, C7P.-, D7.A, D8.A, R5P.1
- net N$46: now also IC5.PG, J17.1, R8B.2; no longer C1P1.+, D13.K, D14.K, J1.4
- net N$47: now also IC5.ILIM, J17.2, R6B.1; no longer C2P1.+, J1.5, R6P1.2
- net N$48: now also IC5.PGFB, J17.3; no longer C4P1.+, R2P1.1, R3P1.2, R4P1.1, R5P1.2
- net PE: no longer J1.1
Other:
- moved on the sheet: C1P1, C2P1, C3P1, C5P1, C6P1, C7P1, D11, D12, D13, D14, R6P1
