File: LT3042_Breakout.brd (EAGLE design)
At the start: 10.7 x 10.7 mm, 2 parts, among them IC1 LT3042, J1 XR2A-0811-N

Commit message: Redid LT3042 breakout
Parts:
- removed IC1: LT3042, Dual Mono Amp Library:SOP50P490X110-11N
- removed J1: XR2A-0811-N, XR2A-0811-N:DIPS762W51P254L1016H390Q8N
- added C18B: 4.7u, Dual Mono Amp Library:CAPC2013X140N
- added C19B: 22u, Dual Mono Amp Library:C1206
- added C20B: 10u, Dual Mono Amp Library:CAPC2012X135N
- added C21B: 0.1u, Dual Mono Amp Library:CAPC2012X135N
- added IC5: LT3042, Dual Mono Amp Library:SOP50P490X110-11N
- added J17: XR2A-0811-N, XR2A-0811-N:DIPS762W51P254L1016H390Q8N
- added R6B: 1k, Dual Mono Amp Library:RESC2012X60N
- added R7B: 33k, Dual Mono Amp Library:R0805
- added R8B: 200k, Dual Mono Amp Library:R0805
Connections:
- removed net N$1: IC1.1, IC1.2, J1.7
- removed net N$2: IC1.3, J1.8
- removed net N$3: IC1.4, J1.1
- removed net N$4: IC1.5, J1.2
- removed net N$5: IC1.10, IC1.9, J1.6
- removed net N$6: IC1.11, IC1.8, IC1.P$1, IC1.P$2, IC1.P$3, IC1.P$4, IC1.P$5, IC1.P$6, J1.5
- removed net N$7: IC1.7, J1.4
- removed net N$8: IC1.6, J1.3
- new net +5V/L/2: C18B.1, IC5.10, IC5.9, J17.6
- new net DGND/2: C18B.2, C19B.2, C19B.DGND, C20B.2, C21B.2, IC5.11, IC5.8, IC5.P$1, IC5.P$2, IC5.P$3, IC5.P$4, IC5.P$5, IC5.P$6, J17.5, R6B.2, R7B.2
- new net N$103: C19B.1, IC5.7, J17.4, R7B.1
- new net N$46: IC5.4, J17.1, R8B.2
- new net N$47: IC5.5, J17.2, R6B.1
- new net N$48: IC5.6, J17.3
- new net VCC/2: C20B.1, C21B.1, IC5.1, IC5.2, IC5.3, J17.7, J17.8, R8B.1
Routing:
- net VCC/2: track 0.00 -> 11.0 mm
- net N$103: track 0.00 -> 10.3 mm
- net N$46: track 0.00 -> 7.25 mm
- net N$47: track 0.00 -> 6.02 mm
- net N$2: track 4.82 -> 0.00 mm
- net N$7: track 4.32 -> 0.00 mm
- net N$3: track 4.32 -> 0.00 mm
- net +5V/L/2: track 0.00 -> 3.24 mm
- net N$8: track 3.20 -> 0.00 mm
- net N$4: track 3.20 -> 0.00 mm
- net N$48: track 0.00 -> 3.14 mm
- added copper zone on layer 16, net +5V/L/2
- added copper zone on layer 1, net DGND/2
- added copper zone on layer 16, net DGND/2
- added copper zone on layer 16, net VCC/2
- removed copper zone on layer 1, net N$1
- removed copper zone on layer 1, net N$5
- removed copper zone on layer 1, net N$6
- removed copper zone on layer 16, net N$6
Other:
- board outline removed
