File: AK4493-Combi9.brd (EAGLE design)
At the start: 237.4 x 160.6 mm, 136 parts, among them IC1 LT3042, IC2 LT3042, IC3 LM317MQDCYR, IC5 LT3042, J1 XR2A-0811-N, J17 XR2A-0811-N, J3 SJ-63033A, J5 XR2A-0811-N, J6 1935255, U1 LM317MTG, U2 LM317MTG

Commit message: Progress
Parts:
- moved R6P1 298.7 mm to (72.6, 100.5)
- moved C5P1 297.6 mm to (84.7, 127.8), turned to 180 degrees
- moved C6P1 275.5 mm to (84.7, 111.1), turned to 180 degrees
- moved C3P1 261.2 mm to (60.4, 127.8)
- moved C7P1 260.5 mm to (60.4, 111.1)
- moved C2P1 242.6 mm to (84.7, 90.0), turned to 180 degrees
- moved C1P1 242.2 mm to (67.9, 90.0), turned to 180 degrees
- moved SH2 150.8 mm to (59.0, 3.00), turned to 180 degrees
- moved D11 2.77 mm to (74.5, 72.9)
- moved D12 2.77 mm to (74.5, 78.9)
- moved D13 2.77 mm to (97.5, 78.9)
- moved D14 2.77 mm to (97.5, 72.9)
Routing:
- net N$57: track 0.00 -> 91.2 mm
- net 6.3_VAC_BLU/2: track 0.00 -> 73.5 mm
- net VCC/2: track 45.1 -> 114.2 mm
- net N$58: track 0.00 -> 64.1 mm
- net 6.3_VAC_GRN/2: track 0.00 -> 60.5 mm
- net 66.3VAC/BRN/2: track 169.6 -> 144.1 mm
- net AGND/2: track 0.00 -> 9.25 mm
- net 115_VAC_BLK/2: track 28.7 -> 37.8 mm
- net +240VDC/2: track 261.5 -> 260.5 mm
Other:
- outline, holes or cut-outs redrawn

Commit message: Progress
Parts:
- added J7: 1935200, Dual Mono Amp Library:1935200
- moved IC3 385.4 mm to (62.3, 174.4), flipped to the bottom, turned to 180 degrees
- moved R6B 116.2 mm to (106.7, 106.7), turned to 90 degrees
- moved R7B 116.0 mm to (106.8, 101.6), turned to 90 degrees
- moved C19B 114.1 mm to (105.4, 97.6), turned to 0 degrees
- moved J17 112.3 mm to (103.9, 108.3), turned to 0 degrees
- moved R8B 111.4 mm to (102.9, 111.2), turned to 180 degrees
- moved IC5 106.5 mm to (100.1, 104.5), turned to 270 degrees
- moved R6D 104.2 mm to (84.3, 149.1), turned to 90 degrees
- moved C20B 103.2 mm to (97.0, 111.2), turned to 180 degrees
- moved R7D 103.0 mm to (84.4, 144.0), turned to 90 degrees
- moved J1 100.7 mm to (81.4, 150.7), turned to 0 degrees
- moved R8D 100.5 mm to (80.5, 153.6), turned to 180 degrees
- moved C19D 100.3 mm to (83.0, 140.0), turned to 0 degrees
- moved C21B 97.4 mm to (93.4, 107.5), turned to 270 degrees
- moved C18B 97.0 mm to (93.4, 102.4), turned to 270 degrees
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Connections:
- removed net +3V3: C18A.1, C26A.1, IC2.10, IC2.9, J5.6, LDO7.1, LDO7.3
- removed net +5V/1: C18D.1, IC1.10, IC1.9, J1.6
- removed net +5V/2: C18B.1, IC5.10, IC5.9, J17.6
- removed net N$65: C27A.1, C28A.1, LDO7.5
- new net +1V8/2: C27A.1, C28A.1, J7.5, LDO7.5
- new net +3V3/2: C18A.1, C26A.1, IC2.10, IC2.9, J5.6, J7.4, LDO7.1, LDO7.3
- new net +5V/L/1: C18D.1, IC1.10, IC1.9, J1.6, J7.2
- new net +5V/L/2: C18B.1, IC5.10, IC5.9, J17.6, J7.3
- new net +5V/L/3: C20A.1, C21A.1, IC2.1, IC2.2, IC2.3, IC3.2, IC3.4, J5.7, J5.8, J7.1, R8A.1
- net DGND/2: now also J7.6
- net VCC/2: now also IC3.3; no longer C20A.1, C21A.1, IC2.1, IC2.2, IC2.3, J5.7, J5.8, R8A.1
Routing:
- net VCC/2: track 114.2 -> 193.3 mm
- net +5V/L/3: track 0.00 -> 11.1 mm
- net +5V/L/2: track 0.00 -> 2.88 mm
- net +5V/L/1: track 0.00 -> 2.88 mm
- net +5V/2: track 2.88 -> 0.00 mm
- net +5V/1: track 2.88 -> 0.00 mm
- net +3V3/2: track 0.00 -> 2.88 mm
- net +3V3: track 2.88 -> 0.00 mm
- added copper zone on layer 16, net +3V3/2
- added copper zone on layer 16, net +5V/L/1
- added copper zone on layer 16, net +5V/L/2
- added copper zone on layer 16, net +5V/L/3
- removed copper zone on layer 16, net +3V3
- removed copper zone on layer 16, net +5V/1
- removed copper zone on layer 16, net +5V/2
Other:
- board size 237.4 x 160.6 mm -> 237.4 x 179 mm

Commit message: Progress
Parts:
- moved LDO7 299.7 mm to (81.0, 167.0), flipped to the bottom
- moved C26A 298.3 mm to (75.0, 168.0), flipped to the bottom
- moved C27A 298.3 mm to (75.0, 165.0), flipped to the bottom
- moved C28A 298.3 mm to (75.0, 162.0), flipped to the bottom
- moved IC3 50.4 mm to (93.4, 134.7), turned to 90 degrees
- moved C18D 38.7 mm to (95.4, 114.8)
- moved C19D 38.7 mm to (107.4, 110.0)
- moved C21D 38.7 mm to (95.4, 119.9)
- moved IC1 38.7 mm to (102.1, 116.9)
- moved R6D 38.7 mm to (108.7, 119.1)
- moved R7D 38.7 mm to (108.8, 114.0)
- moved C20D 38.7 mm to (99.0, 123.6)
- moved J1 38.7 mm to (105.9, 120.7)
- moved R8D 38.7 mm to (104.9, 123.6)
- moved C21A 20.5 mm to (70.9, 149.8)
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Connections:
- net +1V8/2: now also J7.1; no longer J7.5
- net +3V3/2: now also J7.2; no longer J7.4
- net +5V/L/1: now also J7.4; no longer J7.2
- net +5V/L/2: now also J7.5; no longer J7.3
- net +5V/L/3: now also J7.3; no longer J7.1
Routing:
- net +5V/L/2: track 2.88 -> 67.1 mm
- net +5V/L/1: track 2.88 -> 52.7 mm
- net +5V/L/3: track 11.1 -> 52.4 mm
- net VCC/2: track 193.3 -> 164.0 mm
- net +3V3/2: track 2.88 -> 22.8 mm
- net 115_VAC_RED/2: track 53.6 -> 68.8 mm
- net N$58: track 64.1 -> 63.5 mm
- added copper zone on layer 16, net AGND/1
- added copper zone on layer 16, net AGND/2
- removed copper zone on layer 16, net DGND/1
Other:
- board size 237.4 x 179 mm -> 237.4 x 170.5 mm

Commit message: Redid LT3042 breakout
Routing:
- net +240VDC/1: track 0.00 -> 224.5 mm
- net 66.3VAC/ORG/1: track 0.00 -> 199.0 mm
- net N$22: track 100.6 -> 40.9 mm
- added copper zone on layer 16, net DGND/1
Other:
- outline, holes or cut-outs redrawn

Commit message: Progress
Parts:
- added C18B2, C18B4, C18B6: 4.7u, Dual Mono Amp Library:CAPC2013X140N
- added C19B2, C19B4, C19B6: 22u, Dual Mono Amp Library:C1206
- added C1P2, C1P3, C2P2, C2P3, C3P2, C3P3, C5P2, C5P3, C6P2, C6P3, C7P2, C7P3: 68u, 500HXW68MEFR14.5X45:CAPPRD750W80D1475H4700
- added C20B2, C20B4, C20B6: 10u, Dual Mono Amp Library:CAPC2012X135N
- added C21B2, C21B4, C21B6: 0.1u, Dual Mono Amp Library:CAPC2012X135N
- added C26A1, C27A1: 4.7u, Ceramic Capacitor X7R, Dual Mono Amp Library:CAPC2013X140N
- added C28A1: 0.1u, Ceramic Capacitor X7R, Dual Mono Amp Library:CAPC2012X135N
- added C4P1: UCY2E220MPD1TD, UCY2E220MPD1TD:CAPPRD500W60D1025H1750
- added D15, D16, D17, D18, D19, D20, D21, D22: 1N4007FFG, 1N4007FFG:DIOAD1405W86L465D235
- added IC10, IC6, IC8: LT3042, Dual Mono Amp Library:SOP50P490X110-11N
- added IC4: LM317MQDCYR, Dual Mono Amp Library:SOT230P700X180-4N
- added J10, J12, J8: XR2A-0811-N, XR2A-0811-N:DIPS762W51P254L1016H390Q8N
- added J4: 1935255, Dual Mono Amp Library:1935255
- added J9: 1935200, Dual Mono Amp Library:1935200
- added LDO1: LP5907-1.8V, Dual Mono Amp Library:SOT95P280X145-5N
- added R2P1, R3P1: 220, rcl:0411/15
- added R4P1: 300k, rcl:0411/15
- added R5P1: 100k, rcl:0411/15
- added R6B2, R6B4, R6B6: 1k, Dual Mono Amp Library:RESC2012X60N
- added R6P2, R6P3: 330, rcl:0411/15
- added R7B2, R7B4, R7B6: 33k, Dual Mono Amp Library:R0805
- added R8B2, R8B4, R8B6: 200k, Dual Mono Amp Library:R0805
- added SH1: SHORTA5, Dual Mono Amp Library:SHORT_ALL-50
Connections:
- new net +1V8/1: C27A1.1, C28A1.1, J9.1, LDO1.5
- new net +3V3/1: C18B6.1, IC10.10, IC10.9, J12.6, J9.2
- new net +5V/R/1: C18B4.1, IC8.10, IC8.9, J10.6, J9.4
- new net +5V/R/2: C18B2.1, IC6.10, IC6.9, J8.6, J9.5
- new net +5V/R/3: IC4.2, IC4.4, J9.3
- new net 115_VAC_BLK/1: D15.1, D18.2, J4.2
- new net 115_VAC_RED/1: D16.1, D17.2, J4.3
- new net 6.3_VAC_BLU/1: D19.1, D22.2, J4.8
- new net 6.3_VAC_GRN/1: D20.1, D21.2, J4.9
- new net DGND/1: C18B2.2, C18B4.2, C18B6.2, C19B2.2, C19B2.DGND, C19B4.2, C19B4.DGND, C19B6.2, C19B6.DGND, C1P3.2, C20B2.2, C20B4.2, C20B6.2, C21B2.2, C21B4.2, C21B6.2, C26A1.2, C27A1.2, C28A1.2, C2P3.2, C3P3.2, C5P3.2, C6P3.2, C7P3.2, D19.2, D20.2, IC10.11, IC10.8, IC10.P$1, IC10.P$2, IC10.P$3, IC10.P$4, IC10.P$5, IC10.P$6, IC6.11, IC6.8, IC6.P$1, IC6.P$2, IC6.P$3, IC6.P$4, IC6.P$5, IC6.P$6, IC8.11, IC8.8, IC8.P$1, IC8.P$2, IC8.P$3, IC8.P$4, IC8.P$5, IC8.P$6, J10.5, J12.5, J8.5, J9.6, LDO1.2, LDO1.DGND, LDO1.DGND2, LDO1.DGND3, R6B2.2, R6B4.2, R6B6.2, R7B2.2, R7B4.2, R7B6.2, SH1.1
- new net N$59: C1P2.1, D17.1, D18.1, J4.4
- new net N$60: C2P2.1, J4.5, R6P2.2
- new net N$61: C4P1.1, R2P1.1, R3P1.2, R4P1.1, R5P1.2
- new net N$62: C1P3.1, D21.1, D22.1, J4.10
- new net N$63: IC6.4, J8.1, R8B2.2
- new net N$64: C19B2.1, IC6.7, J8.4, R7B2.1
- new net N$65: IC6.5, J8.2, R6B2.1
- new net N$66: IC6.6, J8.3
- new net N$67: C2P3.1, J4.11, R6P3.2
- new net N$71: IC8.4, J10.1, R8B4.2
- new net N$72: C19B4.1, IC8.7, J10.4, R7B4.1
- new net N$73: IC8.5, J10.2, R6B4.1
- new net N$74: IC8.6, J10.3
- new net N$79: IC10.4, J12.1, R8B6.2
- new net N$80: C19B6.1, IC10.7, J12.4, R7B6.1
- new net N$81: IC10.5, J12.2, R6B6.1
- new net N$82: IC10.6, J12.3
- new net VCC/1: C20B2.1, C20B4.1, C20B6.1, C21B2.1, C21B4.1, C21B6.1, C3P3.1, C5P3.1, C6P3.1, C7P3.1, IC10.1, IC10.2, IC10.3, IC4.3, IC6.1, IC6.2, IC6.3, IC8.1, IC8.2, IC8.3, J10.7, J10.8, J12.7, J12.8, J8.7, J8.8, R6P3.1, R8B2.1, R8B4.1, R8B6.1
- net +240VDC/1: now also C3P2.1, C5P2.1, C6P2.1, C7P2.1, R4P1.2, R6P2.1
- net +3V3/2: now also C26A1.1, LDO1.1, LDO1.3
- net 66.3VAC/BRN/1: now also J4.7, R3P1.1
- net 66.3VAC/ORG/1: now also J4.6, R2P1.2
- net AGND/1: now also C1P2.2, C2P2.2, C3P2.2, C4P1.2, C5P2.2, C6P2.2, C7P2.2, D15.2, D16.2, R5P1.1, SH1.2
- net PE: now also J4.1
Routing:
- net VCC/1: track 0.00 -> 33.1 mm
- net N$80: track 0.00 -> 10.3 mm
- net N$72: track 0.00 -> 10.3 mm
- net N$64: track 0.00 -> 10.3 mm
- net N$79: track 0.00 -> 7.25 mm
- net N$63: track 0.00 -> 7.25 mm
- net N$71: track 0.00 -> 7.25 mm
- net N$65: track 0.00 -> 6.02 mm
- net N$81: track 0.00 -> 6.02 mm
- net N$73: track 0.00 -> 6.02 mm
- net +5V/R/2: track 0.00 -> 3.24 mm
- net +5V/R/1: track 0.00 -> 3.24 mm
- net +3V3/1: track 0.00 -> 3.24 mm
- net N$66: track 0.00 -> 3.14 mm
- net N$82: track 0.00 -> 3.14 mm
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
Commit message: Progress
Connections:
- net +3V3/1: now also C26A1.1, LDO1.1, LDO1.3
- net +3V3/2: now also J7.3; no longer C26A1.1, J7.2, LDO1.1, LDO1.3
- net +5V/L/3: now also J7.2; no longer J7.3
Routing:
- net +5V/L/3: track 52.4 -> 66.3 mm
- net +3V3/2: track 22.8 -> 17.8 mm
