File: AK4493-Combi9.brd (EAGLE design)
At the start: 237.4 x 170.5 mm, 199 parts, among them IC1 LT3042, IC10 LT3042, IC2 LT3042, IC3 LM317MQDCYR, IC4 LM317MQDCYR, IC5 LT3042, IC6 LT3042, IC8 LT3042, J1 XR2A-0811-N, J10 XR2A-0811-N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

Commit message: Progress
Parts:
- moved R6P3 204.9 mm to (-72.6, 100.5), turned to 180 degrees
- moved D19 193.0 mm to (-74.5, 72.9)
- moved D20 191.1 mm to (-74.5, 78.9)
- moved D22 188.6 mm to (-97.5, 72.9)
- moved D21 182.5 mm to (-97.5, 78.9)
- moved C3P3 181.7 mm to (-60.4, 127.8), turned to 180 degrees
- moved C6P3 171.9 mm to (-84.7, 111.1)
- moved C7P3 169.6 mm to (-60.4, 111.1), turned to 180 degrees
- moved C5P3 165.3 mm to (-84.7, 127.8)
- moved R4P1 155.6 mm to (-60.4, 56.9), turned to 90 degrees
- moved R5P1 148.6 mm to (-67.2, 56.9), turned to 270 degrees
- moved R6P2 141.5 mm to (-88.2, 31.8), turned to 180 degrees
- moved R2P1 139.4 mm to (-67.2, 23.4), turned to 270 degrees
- moved R3P1 133.5 mm to (-60.4, 23.4), turned to 90 degrees
- moved C1P3 130.9 mm to (-67.9, 90.0)
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Connections:
- net +3V3/1: now also J9.4; no longer J9.5
- net +5V/R/3: now also J9.5; no longer J9.4
Routing:
- net VCC/1: track 33.1 -> 186.4 mm
- net 66.3VAC/BRN/1: track 0.00 -> 95.4 mm
- net N$62: track 0.00 -> 91.2 mm
- net 6.3_VAC_BLU/1: track 0.00 -> 73.5 mm
- net 115_VAC_RED/1: track 0.00 -> 68.8 mm
- net +5V/R/2: track 3.24 -> 70.3 mm
- net N$67: track 0.00 -> 63.5 mm
- net 66.3VAC/ORG/1: track 199.0 -> 260.3 mm
- net +5V/R/3: track 0.00 -> 61.0 mm
- net 6.3_VAC_GRN/1: track 0.00 -> 60.5 mm
- net +5V/R/1: track 3.24 -> 55.8 mm
- net N$60: track 0.00 -> 38.5 mm
- net 115_VAC_BLK/1: track 0.00 -> 37.8 mm
- net +240VDC/1: track 224.5 -> 260.0 mm
- net N$61: track 0.00 -> 32.1 mm
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- added copper zone on layer 16, net +3V3/1
- added copper zone on layer 16, net +5V/R/1
- added copper zone on layer 16, net +5V/R/2
Other:
- board text removed: "115 VAC BLK"
- board text removed: "115 VAC RED"
- board text removed: "6.3 VAC BLU"
- board text removed: "6.3 VAC BRN"
- board text removed: "6.3 VAC GRN"
- board text removed: "6.3 VAC ORG"
- board text removed: "PE"

Commit message: Progress
Parts:
- turned IC4 to 270 degrees
Routing:
- net VCC/1: track 186.4 -> 226.6 mm
- net +5V/R/3: track 61.0 -> 53.3 mm
- net +5V/R/2: track 70.3 -> 64.9 mm
- net +3V3/1: track 21.1 -> 16.0 mm
- net +5V/R/1: track 55.8 -> 52.8 mm
- net +5V/L/3: track 66.3 -> 68.0 mm
- added copper zone on layer 16, net VCC/1

Commit message: Progress
Parts:
- added C5, C6, C7, C8: TCM1A106M8R, Dual Mono Amp Library:CAPPM168X90N
- IC3, IC4: value LM317MQDCYR -> LM1117MPX-5.0_NOPB
- moved C26A 7.62 mm to (72.0, 161.0), turned to 270 degrees
- moved C28A1 7.49 mm to (-68.0, 165.5), turned to 270 degrees
- moved C27A 7.02 mm to (68.0, 165.5), turned to 270 degrees
- moved C26A1 6.32 mm to (-72.0, 161.0), turned to 270 degrees
- moved LDO1 5.37 mm to (-77.6, 165.0), turned to 90 degrees
- moved C28A 4.60 mm to (72.0, 165.5), turned to 270 degrees
- moved LDO7 3.91 mm to (77.6, 165.0), turned to 90 degrees
- moved C27A1 2.49 mm to (-72.0, 165.5), turned to 270 degrees
- moved IC3 0.64 mm to (92.8, 134.7)
- moved IC4 0.64 mm to (-92.8, 134.7)
Connections:
- net +5V/L/3: now also C8.1
- net +5V/R/3: now also C5.1
- net DGND/1: now also C5.2, C6.2, IC4.1
- net DGND/2: now also C7.2, C8.2, IC3.1
- net VCC/1: now also C6.1
- net VCC/2: now also C7.1
Routing:
- net +3V3/2: track 17.8 -> 49.7 mm
- net +3V3/1: track 16.0 -> 47.9 mm
- net +1V8/1: track 0.00 -> 14.8 mm
- net +1V8/2: track 0.00 -> 10.0 mm
- net +5V/L/3: track 68.0 -> 73.5 mm
- net +5V/R/3: track 53.3 -> 58.7 mm
- net VCC/2: track 163.9 -> 167.8 mm
