File: AK4493-Combi9.sch (EAGLE design)
At the start: 136 parts, among them IC1 LT3042, IC2 LT3042, IC3 LM317MQDCYR, IC5 LT3042, J1 XR2A-0811-N, J17 XR2A-0811-N, J3 SJ-63033A, J5 XR2A-0811-N, J6 1935255, U1 LM317MTG, U2 LM317MTG

Commit message: Progress
Parts:
- added J7: 1935200, Dual Mono Amp Library:1935200
Connections:
- removed net +3V3: C18A.1, C26A.1, IC2.OUT, IC2.OUTS, J5.6, LDO7.EN, LDO7.VIN
- removed net +5V/1: C18D.1, IC1.OUT, IC1.OUTS, J1.6
- removed net +5V/2: C18B.1, IC5.OUT, IC5.OUTS, J17.6
- removed net N$65: C27A.1, C28A.1, LDO7.VOUT
- new net +1V8/2: C27A.1, C28A.1, J7.5, LDO7.VOUT
- new net +3V3/2: C18A.1, C26A.1, IC2.OUT, IC2.OUTS, J5.6, J7.4, LDO7.EN, LDO7.VIN
- new net +5V/L/1: C18D.1, IC1.OUT, IC1.OUTS, J1.6, J7.2
- new net +5V/L/2: C18B.1, IC5.OUT, IC5.OUTS, J17.6, J7.3
- new net +5V/L/3: C20A.1, C21A.1, IC2.EN/UV, IC2.IN, IC3.OUT, J5.7, J5.8, J7.1, R8A.1
- net DGND/2: now also J7.6
- net VCC/2: now also IC3.IN; no longer C20A.1, C21A.1, IC2.EN/UV, IC2.IN, J5.7, J5.8, R8A.1
Other:
- moved on the sheet: C18A, C18B, C18D, C19A, C19B, C19D, C20A, C20B, C20D, C21A, C21B, C21D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

Commit message: Progress
Connections:
- net +1V8/2: now also J7.1; no longer J7.5
- net +3V3/2: now also J7.2; no longer J7.4
- net +5V/L/1: now also J7.4; no longer J7.2
- net +5V/L/2: now also J7.5; no longer J7.3
- net +5V/L/3: now also J7.3; no longer J7.1
Changed lines of the file:
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@@
 <attribute name="VALUE" x="324.485" y="167.767" size="1.778" layer="96" rot="R270"/>
 </instance>
-<instance part="SUPPLY9" gate="G$1" x="335.28" y="170.18" smashed="yes" rot="R180">
-<attribute name="VALUE" x="335.915" y="166.37" size="1.778" layer="96" rot="R270"/>
+<instance part="SUPPLY9" gate="G$1" x="330.2" y="170.18" smashed="yes" rot="R180">
+<attribute name="VALUE" x="330.835" y="166.37" size="1.778" layer="96" rot="R270"/>
 </instance>
-<instance part="SUPPLY14" gate="G$1" x="332.74" y="170.18" smashed="yes" rot="R180">
+<instance part="SUPPLY14" gate="G$1" x="327.66" y="170.18" smashed="yes" rot="R180">
+<attribute name="VALUE" x="328.295" y="166.37" size="1.778" layer="96" rot="R270"/>
+</instance>
+<instance part="SUPPLY15" gate="G$1" x="332.74" y="170.18" smashed="yes" rot="R180">
 <attribute name="VALUE" x="333.375" y="166.37" size="1.778" layer="96" rot="R270"/>
 </instance>
-<instance part="SUPPLY15" gate="G$1" x="337.82" y="170.18" smashed="yes" rot="R180">
-<attribute name="VALUE" x="338.455" y="166.37" size="1.778" layer="96" rot="R270"/>
+<instance part="+3V4" gate="G$1" x="335.28" y="170.18" smashed="yes" rot="R180">
+<attribute name="VALUE" x="335.28" y="167.64" size="1.778" layer="96" rot="R270"/>
 </instance>
-<instance part="+3V4" gate="G$1" x="330.2" y="167.64" smashed="yes" rot="R180">
-<attribute name="VALUE" x="330.2" y="165.1" size="1.778" layer="96" rot="R270"/>
-</instance>
-<instance part="+3V5" gate="G$1" x="327.66" y="167.64" smashed="yes" rot="R180">
-<attribute name="VALUE" x="327.66" y="165.1" size="1.778" layer="96" rot="R270"/>
+<instance part="+3V5" gate="G$1" x="337.82" y="170.18" smashed="yes" rot="R180">
+<attribute name="VALUE" x="337.82" y="167.64" size="1.778" layer="96" rot="R270"/>
 </instance>
 <instance part="J7" gate="G$1" x="337.82" y="175.26" smashed="yes" rot="MR90">
@@
 </segment>
 <segment>
-<pinref part="J7" gate="G$1" pin="5"/>
+<pinref part="J7" gate="G$1" pin="1"/>
 <pinref part="+3V5" gate="G$1" pin="+1V8/2"/>
-<wire x1="327.66" y1="170.18" x2="327.66" y2="175.26" width="0.1524" layer="91"/>
+<wire x1="337.82" y1="172.72" x2="337.82" y2="175.26" width="0.1524" layer="91"/>
 </segment>
 </net>
@@
 </segment>
 <segment>
-<pinref part="J7" gate="G$1" pin="4"/>
+<pinref part="J7" gate="G$1" pin="2"/>
 <pinref part="+3V4" gate="G$1" pin="+3V3/2"/>
-<wire x1="330.2" y1="170.18" x2="330.2" y2="175.26" width="0.1524" layer="91"/>
+<wire x1="335.28" y1="172.72" x2="335.28" y2="175.26" width="0.1524" layer="91"/>
 </segment>
 </net>
@@
 </segment>
 <segment>
-<pinref part="J7" gate="G$1" pin="3"/>
+<pinref part="J7" gate="G$1" pin="5"/>
 <pinref part="SUPPLY14" gate="G$1" pin="+5V/L/2"/>
-<wire x1="332.74" y1="172.72" x2="332.74" y2="175.26" width="0.1524" layer="91"/>
+<wire x1="327.66" y1="175.26" x2="327.66" y2="172.72" width="0.1524" layer="91"/>
 </segment>
 </net>
@@
 </segment>
 <segment>
-<pinref part="J7" gate="G$1" pin="2"/>
+<pinref part="J7" gate="G$1" pin="4"/>
 <pinref part="SUPPLY9" gate="G$1" pin="+5V/L/1"/>
-<wire x1="335.28" y1="172.72" x2="335.28" y2="175.26" width="0.1524" layer="91"/>
+<wire x1="330.2" y1="175.26" x2="330.2" y2="172.72" width="0.1524" layer="91"/>
 </segment>
 </net>
@@
 <pinref part="SUPPLY13" gate="G$1" pin="+5V/L/3"/>
 <wire x1="548.64" y1="177.8" x2="538.48" y2="177.8" width="0.1524" layer="91"/>
-</segment>
-<segment>
-<pinref part="J7" gate="G$1" pin="1"/>
-<pinref part="SUPPLY15" gate="G$1" pin="+5V/L/3"/>
-<wire x1="337.82" y1="172.72" x2="337.82" y2="175.26" width="0.1524" layer="91"/>
 </segment>
 <segment>
@@
 <pinref part="SUPPLY16" gate="G$1" pin="+5V/L/3"/>
 </segment>
-</net>
+<segment>
+<pinref part="J7" gate="G$1" pin="3"/>
+<pinref part="SUPPLY15" gate="G$1" pin="+5V/L/3"/>
+<wire x1="332.74" y1="175.26" x2="332.74" y2="172.72" width="0.1524" layer="91"/>
+</segment>
+</net>

Commit message: Progress
Parts:
- added C18B2, C18B4, C18B6: 4.7u, Dual Mono Amp Library:EMK212ABJ475KG-T
- added C19B2, C19B4, C19B6: 22u, Dual Mono Amp Library:EMK316BB7226ML-T
- added C1P2, C1P3, C2P2, C2P3, C3P2, C3P3, C5P2, C5P3, C6P2, C6P3, C7P2, C7P3: 68u, 500HXW68MEFR14.5X45:500HXW68MEFR14.5X45
- added C20B2, C20B4, C20B6: 10u, Dual Mono Amp Library:EMK212BB7106KG-T
- added C21B2, C21B4, C21B6: 0.1u, Dual Mono Amp Library:EMF212B7104KGHT
- added C26A1, C27A1: 4.7u, Ceramic Capacitor X7R, Dual Mono Amp Library:EMK212ABJ475KG-T
- added C28A1: 0.1u, Ceramic Capacitor X7R, Dual Mono Amp Library:EMF212B7104KGHT
- added C4P1: UCY2E220MPD1TD, UCY2E220MPD1TD:UCY2E220MPD1TD
- added D15, D16, D17, D18, D19, D20, D21, D22: 1N4007FFG, 1N4007FFG:1N4007FFG
- added IC10, IC6, IC8: LT3042, Dual Mono Amp Library:LT3042
- added IC4: LM317MQDCYR, Dual Mono Amp Library:LM317MQDCYR
- added J10, J12, J8: XR2A-0811-N, XR2A-0811-N:XR2A-0811-N
- added J4: 1935255, Dual Mono Amp Library:1935255
- added J9: 1935200, Dual Mono Amp Library:1935200
- added LDO1: LP5907-1.8V, Dual Mono Amp Library:LP5907-1.8V
- added R2P1, R3P1: 220, rcl:R-US_0411/15
- added R4P1: 300k, rcl:R-US_0411/15
- added R5P1: 100k, rcl:R-US_0411/15
- added R6B2, R6B4, R6B6: 1k, Dual Mono Amp Library:CHP0805-FX-1001ELF
- added R6P2, R6P3: 330, rcl:R-US_0411/15
- added R7B2, R7B4, R7B6: 33k, Dual Mono Amp Library:CPF0805B51KE1
- added R8B2, R8B4, R8B6: 200k, Dual Mono Amp Library:RR1220P-204-D
- added SH1: SHORTA5, Dual Mono Amp Library:SHORTA5
Connections:
- new net +1V8/1: C27A1.1, C28A1.1, J9.1, LDO1.VOUT
- new net +3V3/1: C18B6.1, IC10.OUT, IC10.OUTS, J12.6, J9.2
- new net +5V/R/1: C18B4.1, IC8.OUT, IC8.OUTS, J10.6, J9.4
- new net +5V/R/2: C18B2.1, IC6.OUT, IC6.OUTS, J8.6, J9.5
- new net +5V/R/3: IC4.OUT, J9.3
- new net 115_VAC_BLK/1: D15.K, D18.A, J4.2
- new net 115_VAC_RED/1: D16.K, D17.A, J4.3
- new net 6.3_VAC_BLU/1: D19.K, D22.A, J4.8
- new net 6.3_VAC_GRN/1: D20.K, D21.A, J4.9
- new net DGND/1: C18B2.2, C18B4.2, C18B6.2, C19B2.2, C19B4.2, C19B6.2, C1P3.-, C20B2.2, C20B4.2, C20B6.2, C21B2.2, C21B4.2, C21B6.2, C26A1.2, C27A1.2, C28A1.2, C2P3.-, C3P3.-, C5P3.-, C6P3.-, C7P3.-, D19.A, D20.A, IC10.GND, IC6.GND, IC8.GND, J10.5, J12.5, J8.5, J9.6, LDO1.GND, R6B2.2, R6B4.2, R6B6.2, R7B2.2, R7B4.2, R7B6.2, SH1.P$1
- new net N$59: C1P2.+, D17.K, D18.K, J4.4
- new net N$60: C2P2.+, J4.5, R6P2.2
- new net N$61: C4P1.+, R2P1.1, R3P1.2, R4P1.1, R5P1.2
- new net N$62: C1P3.+, D21.K, D22.K, J4.10
- new net N$63: IC6.PG, J8.1, R8B2.2
- new net N$64: C19B2.1, IC6.SET, J8.4, R7B2.1
- new net N$65: IC6.ILIM, J8.2, R6B2.1
- new net N$66: IC6.PGFB, J8.3
- new net N$67: C2P3.+, J4.11, R6P3.2
- new net N$71: IC8.PG, J10.1, R8B4.2
- new net N$72: C19B4.1, IC8.SET, J10.4, R7B4.1
- new net N$73: IC8.ILIM, J10.2, R6B4.1
- new net N$74: IC8.PGFB, J10.3
- new net N$79: IC10.PG, J12.1, R8B6.2
- new net N$80: C19B6.1, IC10.SET, J12.4, R7B6.1
- new net N$81: IC10.ILIM, J12.2, R6B6.1
- new net N$82: IC10.PGFB, J12.3
- new net VCC/1: C20B2.1, C20B4.1, C20B6.1, C21B2.1, C21B4.1, C21B6.1, C3P3.+, C5P3.+, C6P3.+, C7P3.+, IC10.EN/UV, IC10.IN, IC4.IN, IC6.EN/UV, IC6.IN, IC8.EN/UV, IC8.IN, J10.7, J10.8, J12.7, J12.8, J8.7, J8.8, R6P3.1, R8B2.1, R8B4.1, R8B6.1
- net +240VDC/1: now also C3P2.+, C5P2.+, C6P2.+, C7P2.+, R4P1.2, R6P2.1
- net +3V3/2: now also C26A1.1, LDO1.EN, LDO1.VIN
- net 66.3VAC/BRN/1: now also J4.7, R3P1.1
- net 66.3VAC/ORG/1: now also J4.6, R2P1.2
- net AGND/1: now also C1P2.-, C2P2.-, C3P2.-, C4P1.-, C5P2.-, C6P2.-, C7P2.-, D15.A, D16.A, R5P1.1, SH1.P$2
- net PE: now also J4.1

Commit message: Progress
Connections:
- net +3V3/1: now also C26A1.1, LDO1.EN, LDO1.VIN
- net +3V3/2: now also J7.3; no longer C26A1.1, J7.2, LDO1.EN, LDO1.VIN
- net +5V/L/3: now also J7.2; no longer J7.3
Changed lines of the file:
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@@
 <part name="C27A1" library="Dual Mono Amp Library" deviceset="EMK212ABJ475KG-T" device="" value="4.7u, Ceramic Capacitor X7R"/>
 <part name="IC4" library="Dual Mono Amp Library" library_urn="urn:adsk.eagle:library:47621477" deviceset="LM317MQDCYR" device="" package3d_urn="urn:adsk.eagle:package:47621665/2"/>
-<part name="+3V6" library="Dual Mono Amp Library" library_urn="urn:adsk.eagle:library:47621477" deviceset="+3V3/2" device=""/>
 <part name="J9" library="Dual Mono Amp Library" library_urn="urn:adsk.eagle:library:47621477" deviceset="1935200" device="" package3d_urn="urn:adsk.eagle:package:50913441/1"/>
 <part name="SUPPLY33" library="Dual Mono Amp Library" library_urn="urn:adsk.eagle:library:47621477" deviceset="+5V/R/1" device=""/>
@@
 <part name="+3V8" library="Dual Mono Amp Library" library_urn="urn:adsk.eagle:library:47621477" deviceset="+3V3/1" device=""/>
 <part name="+3V9" library="Dual Mono Amp Library" library_urn="urn:adsk.eagle:library:47621477" deviceset="+1V8/1" device=""/>
+<part name="+3V11" library="Dual Mono Amp Library" library_urn="urn:adsk.eagle:library:47621477" deviceset="+3V3/1" device=""/>
 </parts>
 <sheets>
@@
 <attribute name="VALUE" x="328.295" y="166.37" size="1.778" layer="96" rot="R270"/>
 </instance>
-<instance part="SUPPLY15" gate="G$1" x="332.74" y="170.18" smashed="yes" rot="R180">
-<attribute name="VALUE" x="333.375" y="166.37" size="1.778" layer="96" rot="R270"/>
+<instance part="SUPPLY15" gate="G$1" x="335.28" y="170.18" smashed="yes" rot="R180">
+<attribute name="VALUE" x="335.915" y="166.37" size="1.778" layer="96" rot="R270"/>
 </instance>
-<instance part="+3V4" gate="G$1" x="335.28" y="170.18" smashed="yes" rot="R180">
-<attribute name="VALUE" x="335.28" y="167.64" size="1.778" layer="96" rot="R270"/>
+<instance part="+3V4" gate="G$1" x="332.74" y="170.18" smashed="yes" rot="R180">
+<attribute name="VALUE" x="332.74" y="167.64" size="1.778" layer="96" rot="R270"/>
 </instance>
 <instance part="+3V5" gate="G$1" x="337.82" y="170.18" smashed="yes" rot="R180">
@@
 <attribute name="VALUE" x="-533.4" y="167.64" size="1.778" layer="96" rot="MR0"/>
 </instance>
-<instance part="+3V6" gate="G$1" x="-462.28" y="165.1" smashed="yes" rot="MR270">
-<attribute name="VALUE" x="-457.2" y="167.64" size="1.778" layer="96" rot="MR0"/>
-</instance>
 <instance part="J9" gate="G$1" x="-337.82" y="175.26" smashed="yes" rot="R90">
 <attribute name="NAME" x="-345.44" y="191.77" size="1.778" layer="95" rot="R90" align="center-left"/>
@@
 <attribute name="VALUE" x="-335.28" y="175.26" size="1.778" layer="96" rot="R270"/>
 </instance>
+<instance part="+3V11" gate="G$1" x="-462.28" y="165.1" smashed="yes" rot="R90">
+<attribute name="VALUE" x="-457.2" y="162.56" size="1.778" layer="96" rot="R180"/>
+</instance>
 </instances>
 <busses>
@@
 </segment>
 <segment>
-<pinref part="J7" gate="G$1" pin="2"/>
 <pinref part="+3V4" gate="G$1" pin="+3V3/2"/>
-<wire x1="335.28" y1="172.72" x2="335.28" y2="175.26" width="0.1524" layer="91"/>
-</segment>
-<segment>
-<pinref part="LDO1" gate="G$1" pin="EN"/>
-<wire x1="-454.66" y1="170.18" x2="-457.2" y2="170.18" width="0.1524" layer="91"/>
-<wire x1="-457.2" y1="170.18" x2="-457.2" y2="165.1" width="0.1524" layer="91"/>
-<pinref part="LDO1" gate="G$1" pin="VIN"/>
-<wire x1="-457.2" y1="165.1" x2="-454.66" y2="165.1" width="0.1524" layer="91"/>
-<wire x1="-457.2" y1="165.1" x2="-459.74" y2="165.1" width="0.1524" layer="91"/>
-<junction x="-457.2" y="165.1"/>
-<pinref part="C26A1" gate="G$1" pin="1"/>
-<wire x1="-457.2" y1="162.56" x2="-457.2" y2="165.1" width="0.1524" layer="91"/>
-<pinref part="+3V6" gate="G$1" pin="+3V3/2"/>
+<pinref part="J7" gate="G$1" pin="3"/>
+<wire x1="332.74" y1="172.72" x2="332.74" y2="175.26" width="0.1524" layer="91"/>
 </segment>
 </net>
@@
 </segment>
 <segment>
-<pinref part="J7" gate="G$1" pin="3"/>
 <pinref part="SUPPLY15" gate="G$1" pin="+5V/L/3"/>
-<wire x1="332.74" y1="175.26" x2="332.74" y2="172.72" width="0.1524" layer="91"/>
+<pinref part="J7" gate="G$1" pin="2"/>
+<wire x1="335.28" y1="172.72" x2="335.28" y2="175.26" width="0.1524" layer="91"/>
 </segment>
 </net>
@@
 <pinref part="+3V8" gate="G$1" pin="+3V3/1"/>
 </segment>
+<segment>
+<pinref part="LDO1" gate="G$1" pin="EN"/>
+<wire x1="-454.66" y1="170.18" x2="-457.2" y2="170.18" width="0.1524" layer="91"/>
+<wire x1="-457.2" y1="170.18" x2="-457.2" y2="165.1" width="0.1524" layer="91"/>
+<pinref part="LDO1" gate="G$1" pin="VIN"/>
+<wire x1="-457.2" y1="165.1" x2="-454.66" y2="165.1" width="0.1524" layer="91"/>
+<wire x1="-457.2" y1="165.1" x2="-459.74" y2="165.1" width="0.1524" layer="91"/>
+<junction x="-457.2" y="165.1"/>
+<pinref part="C26A1" gate="G$1" pin="1"/>
+<wire x1="-457.2" y1="162.56" x2="-457.2" y2="165.1" width="0.1524" layer="91"/>
+<pinref part="+3V11" gate="G$1" pin="+3V3/1"/>
+</segment>
 </net>

Commit message: Progress
Parts:
- J4: device Dual Mono Amp Library:1935255 -> 1935255:1935255
- J9: device Dual Mono Amp Library:1935200 -> 1935200:1935200
Connections:
- net +1V8/1: now also J9.6; no longer J9.1
- net +3V3/1: now also J9.5; no longer J9.2
- net +5V/R/1: now also J9.3; no longer J9.4
- net +5V/R/2: now also J9.2; no longer J9.5
- net +5V/R/3: now also J9.4; no longer J9.3
- net 115_VAC_BLK/1: now also J4.10; no longer J4.2
- net 115_VAC_RED/1: now also J4.9; no longer J4.3
- net 6.3_VAC_BLU/1: now also J4.4; no longer J4.8
- net 6.3_VAC_GRN/1: now also J4.3; no longer J4.9
- net 66.3VAC/BRN/1: now also J4.5; no longer J4.7
- net DGND/1: now also J9.1; no longer J9.6
- net N$59: now also J4.8; no longer J4.4
- net N$60: now also J4.7; no longer J4.5
- net N$62: now also J4.2; no longer J4.10
- net N$67: now also J4.1; no longer J4.11
- net PE: now also J4.11; no longer J4.1
Changed lines of the file:
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@@
 <part name="C6P3" library="500HXW68MEFR14.5X45" deviceset="500HXW68MEFR14.5X45" device="" value="68u"/>
 <part name="C7P3" library="500HXW68MEFR14.5X45" deviceset="500HXW68MEFR14.5X45" device="" value="68u"/>
-<part name="J4" library="Dual Mono Amp Library" library_urn="urn:adsk.eagle:library:47621477" deviceset="1935255" device="" package3d_urn="urn:adsk.eagle:package:50907200/1"/>
 <part name="AGND25" library="Dual Mono Amp Library" library_urn="urn:adsk.eagle:library:47621477" deviceset="AGND/1" device=""/>
 <part name="AGND26" library="Dual Mono Amp Library" library_urn="urn:adsk.eagle:library:47621477" deviceset="AGND/1" device=""/>
@@
 <part name="C27A1" library="Dual Mono Amp Library" deviceset="EMK212ABJ475KG-T" device="" value="4.7u, Ceramic Capacitor X7R"/>
 <part name="IC4" library="Dual Mono Amp Library" library_urn="urn:adsk.eagle:library:47621477" deviceset="LM317MQDCYR" device="" package3d_urn="urn:adsk.eagle:package:47621665/2"/>
-<part name="J9" library="Dual Mono Amp Library" library_urn="urn:adsk.eagle:library:47621477" deviceset="1935200" device="" package3d_urn="urn:adsk.eagle:package:50913441/1"/>
 <part name="SUPPLY33" library="Dual Mono Amp Library" library_urn="urn:adsk.eagle:library:47621477" deviceset="+5V/R/1" device=""/>
 <part name="SUPPLY35" library="Dual Mono Amp Library" library_urn="urn:adsk.eagle:library:47621477" deviceset="+5V/R/2" device=""/>
@@
 <part name="+3V9" library="Dual Mono Amp Library" library_urn="urn:adsk.eagle:library:47621477" deviceset="+1V8/1" device=""/>
 <part name="+3V11" library="Dual Mono Amp Library" library_urn="urn:adsk.eagle:library:47621477" deviceset="+3V3/1" device=""/>
+<part name="J4" library="1935255" deviceset="1935255" device=""/>
+<part name="J9" library="1935200" deviceset="1935200" device=""/>
 </parts>
 <sheets>
@@
 <attribute name="VALUE" x="-252.984" y="65.151" size="1.778" layer="96" rot="MR180"/>
 </instance>
-<instance part="J4" gate="G$1" x="-172.72" y="203.2" smashed="yes" rot="MR90">
-<attribute name="NAME" x="-165.1" y="219.71" size="1.778" layer="95" rot="MR90" align="center-left"/>
-<attribute name="VALUE" x="-167.64" y="219.71" size="1.778" layer="96" rot="MR90" align="center-left"/>
-</instance>
 <instance part="AGND25" gate="G$1" x="-157.48" y="81.28" smashed="yes" rot="R180">
 <attribute name="VALUE" x="-154.94" y="86.36" size="1.778" layer="96" rot="R270"/>
@@
 <attribute name="VALUE" x="-533.4" y="167.64" size="1.778" layer="96" rot="MR0"/>
 </instance>
-<instance part="J9" gate="G$1" x="-337.82" y="175.26" smashed="yes" rot="R90">
-<attribute name="NAME" x="-345.44" y="191.77" size="1.778" layer="95" rot="R90" align="center-left"/>
-<attribute name="VALUE" x="-342.9" y="191.77" size="1.778" layer="96" rot="R90" align="center-left"/>
-</instance>
 <instance part="SUPPLY33" gate="G$1" x="-421.64" y="129.54" smashed="yes">
 <attribute name="VALUE" x="-425.45" y="132.715" size="1.778" layer="96"/>
@@
 <attribute name="VALUE" x="-457.2" y="162.56" size="1.778" layer="96" rot="R180"/>
 </instance>
+<instance part="J4" gate="G$1" x="-198.12" y="203.2" smashed="yes" rot="R90">
+<attribute name="NAME" x="-205.74" y="219.71" size="1.778" layer="95" rot="R90" align="center-left"/>
+<attribute name="VALUE" x="-203.2" y="219.71" size="1.778" layer="96" rot="R90" align="center-left"/>
+</instance>
+<instance part="J9" gate="G$1" x="-325.12" y="175.26" smashed="yes" rot="MR90">
+<attribute name="NAME" x="-317.5" y="191.77" size="1.778" layer="95" rot="MR90" align="center-left"/>
+<attribute name="VALUE" x="-320.04" y="191.77" size="1.778" layer="96" rot="MR90" align="center-left"/>
+</instance>
 </instances>
 <busses>
@@
 <wire x1="-124.46" y1="160.02" x2="-124.46" y2="137.16" width="0.1524" layer="91"/>
 <wire x1="-187.96" y1="203.2" x2="-187.96" y2="170.18" width="0.1524" layer="91"/>
-<pinref part="J4" gate="G$1" pin="7"/>
 <pinref part="U$17" gate="G$1" pin="66.3VAC/BRN/1"/>
+<pinref part="J4" gate="G$1" pin="5"/>
 </segment>
 </net>
@@
 <wire x1="-175.26" y1="160.02" x2="-175.26" y2="127" width="0.1524" layer="91"/>
 <wire x1="-185.42" y1="203.2" x2="-185.42" y2="165.1" width="0.1524" layer="91"/>
-<pinref part="J4" gate="G$1" pin="6"/>
 <pinref part="U$18" gate="G$1" pin="66.3VAC/ORG/1"/>
+<pinref part="J4" gate="G$1" pin="6"/>
 </segment>
 </net>
@@
 <pinref part="PE2" gate="M" pin="PE"/>
 <wire x1="-172.72" y1="200.66" x2="-172.72" y2="203.2" width="0.1524" layer="91"/>
-<pinref part="J4" gate="G$1" pin="1"/>
+<pinref part="J4" gate="G$1" pin="11"/>
 </segment>
 </net>
@@
 <wire x1="-215.9" y1="193.04" x2="-180.34" y2="193.04" width="0.1524" layer="91"/>
 <wire x1="-180.34" y1="193.04" x2="-180.34" y2="203.2" width="0.1524" layer="91"/>
-<pinref part="J4" gate="G$1" pin="4"/>
+<pinref part="J4" gate="G$1" pin="8"/>
 </segment>
 </net>
@@
 <wire x1="-218.44" y1="195.58" x2="-182.88" y2="195.58" width="0.1524" layer="91"/>
 <wire x1="-182.88" y1="195.58" x2="-182.88" y2="203.2" width="0.1524" layer="91"/>
-<pinref part="J4" gate="G$1" pin="5"/>
+<pinref part="J4" gate="G$1" pin="7"/>
 </segment>
 </net>
@@
 <wire x1="-264.16" y1="198.12" x2="-195.58" y2="198.12" width="0.1524" layer="91"/>
 <wire x1="-195.58" y1="198.12" x2="-195.58" y2="203.2" width="0.1524" layer="91"/>
-<pinref part="J4" gate="G$1" pin="10"/>
+<pinref part="J4" gate="G$1" pin="2"/>
 </segment>
 </net>
@@
 <wire x1="-266.7" y1="200.66" x2="-198.12" y2="200.66" width="0.1524" layer="91"/>
 <wire x1="-198.12" y1="200.66" x2="-198.12" y2="203.2" width="0.1524" layer="91"/>
-<pinref part="J4" gate="G$1" pin="11"/>
+<pinref part="J4" gate="G$1" pin="1"/>
 </segment>
 </net>
@@
 <junction x="-256.54" y="147.32"/>
 <wire x1="-228.6" y1="142.24" x2="-256.54" y2="142.24" width="0.1524" layer="91"/>
-<pinref part="J4" gate="G$1" pin="9"/>
+<pinref part="J4" gate="G$1" pin="3"/>
 </segment>
 </net>
@@
 <wire x1="-236.22" y1="172.72" x2="-236.22" y2="167.64" width="0.1524" layer="91"/>
 <wire x1="-190.5" y1="172.72" x2="-236.22" y2="172.72" width="0.1524" layer="91"/>
-<pinref part="J4" gate="G$1" pin="8"/>
+<pinref part="J4" gate="G$1" pin="4"/>
 </segment>
 </net>
@@
 <wire x1="-177.8" y1="203.2" x2="-177.8" y2="142.24" width="0.1524" layer="91"/>
 <label x="-177.8" y="190.5" size="1.27" layer="95" rot="MR0" xref="yes"/>
-<pinref part="J4" gate="G$1" pin="3"/>
+<pinref part="J4" gate="G$1" pin="9"/>
 </segment>
 </net>
@@
 <wire x1="-175.26" y1="203.2" x2="-175.26" y2="167.64" width="0.1524" layer="91"/>
 <label x="-175.26" y="187.96" size="1.27" layer="95" rot="MR0" xref="yes"/>
-<pinref part="J4" gate="G$1" pin="2"/>
+<pinref part="J4" gate="G$1" pin="10"/>
 </segment>
 </net>
@@
 <segment>
 <wire x1="-325.12" y1="175.26" x2="-325.12" y2="172.72" width="0.1524" layer="91"/>
-<pinref part="J9" gate="G$1" pin="6"/>
 <pinref part="SUPPLY20" gate="G$1" pin="DGND/1"/>
+<pinref part="J9" gate="G$1" pin="1"/>
 </segment>
 </net>
@@
 </segment>
 <segment>
-<pinref part="J9" gate="G$1" pin="3"/>
 <wire x1="-332.74" y1="175.26" x2="-332.74" y2="172.72" width="0.1524" layer="91"/>
 <pinref part="SUPPLY19" gate="G$1" pin="+5V/R/3"/>
+<pinref part="J9" gate="G$1" pin="4"/>
 </segment>
 </net>
@@
 </segment>
 <segment>
-<pinref part="J9" gate="G$1" pin="1"/>
 <wire x1="-337.82" y1="172.72" x2="-337.82" y2="175.26" width="0.1524" layer="91"/>
 <pinref part="+3V9" gate="G$1" pin="+1V8/1"/>
+<pinref part="J9" gate="G$1" pin="6"/>
 </segment>
 </net>
@@
 </segment>
 <segment>
-<pinref part="J9" gate="G$1" pin="4"/>
 <wire x1="-330.2" y1="175.26" x2="-330.2" y2="172.72" width="0.1524" layer="91"/>
 <pinref part="SUPPLY18" gate="G$1" pin="+5V/R/1"/>
+<pinref part="J9" gate="G$1" pin="3"/>
 </segment>
 </net>
@@
 </segment>
 <segment>
-<pinref part="J9" gate="G$1" pin="2"/>
 <wire x1="-335.28" y1="172.72" x2="-335.28" y2="175.26" width="0.1524" layer="91"/>
 <pinref part="+3V8" gate="G$1" pin="+3V3/1"/>
+<pinref part="J9" gate="G$1" pin="5"/>
 </segment>
 <segment>
@@
 </segment>
 <segment>
-<pinref part="J9" gate="G$1" pin="5"/>
 <wire x1="-327.66" y1="175.26" x2="-327.66" y2="172.72" width="0.1524" layer="91"/>
 <pinref part="SUPPLY17" gate="G$1" pin="+5V/R/2"/>
+<pinref part="J9" gate="G$1" pin="2"/>
 </segment>
 </net>
