File: AK4493-Combi10.brd (EAGLE design)
At the start: 237.4 x 170.5 mm, 201 parts, among them IC1 LT3042, IC10 LT3042, IC2 LT3042, IC3 LM1117MPX-5.0_NOPB, IC4 LM1117MPX-5.0_NOPB, IC5 LT3042, IC6 LT3042, IC8 LT3042, J1 XR2A-0811-N, J10 XR2A-0811-N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

Commit message: Progress
Parts:
- C1P, C1P1, C1P2, C1P3, C2P, C2P1, C2P2, C2P3, C3P, C3P1, C3P2, C3P3, C5P, C5P1, C5P2, C5P3, C6P, C6P1, C6P2, C6P3, C7P, C7P1, C7P2, C7P3: device 500HXW68MEFR14.5X45:CAPPRD750W80D1475H4700 -> Dual Mono Amp Library:CAPPRD750W80D1475H4700
- D10, D11, D12, D13, D14, D15, D16, D17, D18, D19, D20, D21, D22, D7, D8, D9: device 1N4007FFG:DIOAD1405W86L465D235 -> Dual Mono Amp Library:DIOAD1405W86L465D235
- J4: device 1935255:1935255 -> Dual Mono Amp Library:1935255
- J9: device 1935200:1935200 -> Dual Mono Amp Library:1935200
- moved LDO1 1.90 mm to (-79.5, 165.0)
Routing:
- net +3V3/2: track 49.1 -> 43.9 mm
- net +3V3/1: track 47.0 -> 43.7 mm
- net +1V8/1: track 14.7 -> 17.5 mm
- net DGND/2: track 0.00 -> 2.50 mm
- net DGND/1: track 0.00 -> 2.50 mm
- net +1V8/2: track 18.8 -> 17.5 mm
- added copper zone on layer 16, net +1V8/1
- added copper zone on layer 16, net +1V8/2

Commit message: Progress
Parts:
- C4P, C4P1: device UCY2E220MPD1TD:CAPPRD500W60D1025H1750 -> Dual Mono Amp Library:CAPPRD500W60D1025H1750
- J1, J10, J12, J17, J5, J8: device XR2A-0811-N:DIPS762W51P254L1016H390Q8N -> Dual Mono Amp Library:DIPS762W51P254L1016H390Q8N
- R2P, R2P1, R3P, R3P1, R4P, R4P1, R5P, R5P1, R6P, R6P1, R6P2, R6P3: device rcl:0411/15 -> Dual Mono Amp Library:0411/15

Commit message: Progress
Parts:
- R7A, R7B6: device Dual Mono Amp Library:R0805 -> Dual Mono Amp Library:RESC2012X65N
