File: AK4493-Combi10.sch (EAGLE design)
At the start: 201 parts, among them IC1 LT3042, IC10 LT3042, IC2 LT3042, IC3 LM1117MPX-5.0_NOPB, IC4 LM1117MPX-5.0_NOPB, IC5 LT3042, IC6 LT3042, IC8 LT3042, J1 XR2A-0811-N, J10 XR2A-0811-N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

Commit message: Progress
Parts:
- C1P, C1P1, C1P2, C1P3, C2P, C2P1, C2P2, C2P3, C3P, C3P1, C3P2, C3P3, C5P, C5P1, C5P2, C5P3, C6P, C6P1, C6P2, C6P3, C7P, C7P1, C7P2, C7P3: device 500HXW68MEFR14.5X45:500HXW68MEFR14.5X45 -> Dual Mono Amp Library:500HXW68MEFR14.5X45
- D10, D11, D12, D13, D14, D15, D16, D17, D18, D19, D20, D21, D22, D7, D8, D9: device 1N4007FFG:1N4007FFG -> Dual Mono Amp Library:1N4007FFG
- J4: device 1935255:1935255 -> Dual Mono Amp Library:1935255
- J9: device 1935200:1935200 -> Dual Mono Amp Library:1935200

Commit message: Progress
Parts:
- C4P, C4P1: device UCY2E220MPD1TD:UCY2E220MPD1TD -> Dual Mono Amp Library:UCY2E220MPD1TD
- J1, J10, J12, J17, J5, J8: device XR2A-0811-N:XR2A-0811-N -> Dual Mono Amp Library:XR2A-0811-N
- R2P, R2P1, R3P, R3P1: device rcl:R-US_0411/15 -> Dual Mono Amp Library:PR02000202200JA1000411/15
- R4P, R4P1: device rcl:R-US_0411/15 -> Dual Mono Amp Library:PR02000203003JR5000411/15
- R5P, R5P1: device rcl:R-US_0411/15 -> Dual Mono Amp Library:PR02000201003JA1000411/15
- R6P, R6P1, R6P2, R6P3: device rcl:R-US_0411/15 -> Dual Mono Amp Library:PR02000203300JA1000411/15

Commit message: Progress
Parts:
- R7A, R7B6: device Dual Mono Amp Library:CPF0805B51KE1 -> Dual Mono Amp Library:CPF0805B33KE1
Changed lines of the file:
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@@
 <part name="IC2" library="Dual Mono Amp Library" deviceset="LT3042" device=""/>
 <part name="R6A" library="Dual Mono Amp Library" deviceset="CHP0805-FX-1001ELF" device="" value="1k"/>
-<part name="R7A" library="Dual Mono Amp Library" deviceset="CPF0805B51KE1" device="" value="33k"/>
+<part name="R7A" library="Dual Mono Amp Library" library_urn="urn:adsk.eagle:library:47621477" deviceset="CPF0805B33KE1" device="" package3d_urn="urn:adsk.eagle:package:47621631/2" value="33k"/>
 <part name="R8A" library="Dual Mono Amp Library" deviceset="RR1220P-204-D" device="" value="200k"/>
 <part name="C21A" library="Dual Mono Amp Library" deviceset="EMF212B7104KGHT" device="" value="0.1u"/>
@@
 <part name="IC10" library="Dual Mono Amp Library" deviceset="LT3042" device=""/>
 <part name="R6B6" library="Dual Mono Amp Library" deviceset="CHP0805-FX-1001ELF" device="" value="1k"/>
-<part name="R7B6" library="Dual Mono Amp Library" deviceset="CPF0805B51KE1" device="" value="33k"/>
+<part name="R7B6" library="Dual Mono Amp Library" library_urn="urn:adsk.eagle:library:47621477" deviceset="CPF0805B33KE1" device="" package3d_urn="urn:adsk.eagle:package:47621631/2" value="33k"/>
 <part name="R8B6" library="Dual Mono Amp Library" deviceset="RR1220P-204-D" device="" value="200k"/>
 <part name="C21B6" library="Dual Mono Amp Library" deviceset="EMF212B7104KGHT" device="" value="0.1u"/>
