File: Archive/AK4493-Combi.brd (EAGLE design)
At the start: 178 x 151.3 mm, 224 parts, among them IC1 LT3042, IC2 AK4493, IC3 AK4493, IC4 LT3042, IC4A SN74ABT273DBR, IC5 LT3042, IC6 LT3042, IC7 LT3042, IC8 LT3042, J15 XR2A-0811-N, J16 XR2A-0811-N, J17 XR2A-0811-N, J18 XR2A-0811-N, J19 XR2A-0811-N, J20 XR2A-0811-N, J26 SJ-63033A, J27 1935161, U1 AZ1117H-5.0TRE1, X1 JST-XH-07-PIN-ROUND-PAD, X4 JST-XH-04-PIN-ROUND-PAD

Commit message: Progress
Parts:
- moved TP1 3.45 mm to (42.2, 39.6)
- moved X4 1.68 mm to (59.2, 108.7)
- moved C1A 0.80 mm to (70.6, 117.4)
- moved R10 0.77 mm to (70.8, 122.5)
- moved R20 0.77 mm to (70.8, 125.0)
- moved R5A 0.77 mm to (70.8, 119.9)
- moved C6 0.50 mm to (55.4, 136.4)
- moved C7 0.50 mm to (55.4, 131.4)
- moved D9 0.50 mm to (60.3, 144.5)
- moved R1 0.50 mm to (55.4, 133.9)
- moved U$1 0.50 mm to (59.2, 130.1)
Connections:
- net AGND: no longer IC2.P$11, IC2.P$12, IC2.P$13, IC2.P$14, IC2.P$15, IC2.P$16, IC2.P$19, IC2.P$20, IC2.P$21, IC2.P$22, IC2.P$23, IC2.P$24, IC2.P$3, IC2.P$5, IC2.P$7, IC2.P$9, IC3.P$11, IC3.P$12, IC3.P$13, IC3.P$14, IC3.P$15, IC3.P$16, IC3.P$19, IC3.P$20, IC3.P$21, IC3.P$22, IC3.P$23, IC3.P$24, IC3.P$3, IC3.P$5, IC3.P$7, IC3.P$9
Routing:
- net DIF0: track 173.2 -> 108.7 mm
- net DIF1: track 168.6 -> 110.1 mm
- net +3V3: track 177.7 -> 223.2 mm, vias 6 -> 9
- net DGND: track 0.00 -> 31.4 mm
- net PDN: track 152.9 -> 143.6 mm
- net VCC/1: track 563.3 -> 554.0 mm
- net +5V/3: track 51.9 -> 47.4 mm
- net +5V/4: track 62.7 -> 58.7 mm
- net +240VDC: track 310.4 -> 306.9 mm
- net 66.3VAC/1: track 294.7 -> 291.9 mm
- net +5V/5: track 86.8 -> 84.8 mm
- net +5V/2: track 92.0 -> 90.2 mm
- net ROT_LEDB: track 17.6 -> 16.3 mm
- net N$39: track 83.5 -> 82.3 mm
- net SCL0: track 157.0 -> 155.8 mm
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